Commit message: join with gemini

File: urdf/gemini_335_336.urdf copy.xacro (robot description, xacro)
@@ -1,8 +1,9 @@
 <?xml version="1.0" encoding="utf-8"?>
+<!-- This URDF was automatically created by SolidWorks to URDF Exporter! Originally created by
+Stephen Brawner (brawner@gmail.com)
+     Commit Version: 1.6.0-4-g7f85cfe  Build Version: 1.6.7995.38578
+     For more information, please see http://wiki.ros.org/sw_urdf_exporter -->
 <robot xmlns:xacro="http://ros.org/wiki/xacro" name="gemini_335_336">
-  <!-- proprietà per i mesh -->
-  <xacro:property name="mesh_path" value="package://orbbec_description/meshes/gemini335_336/" />
-  <!-- macro che istanzia il Gemini e lo attacca a un parent -->
-  <xacro:macro name="gemini_335_336" params="parent_link">
+    <xacro:property name="mesh_path" value="package://orbbec_description/meshes/gemini335_336/" />
     <link name="camera_link">
         <inertial>
@@ -54,7 +55,7 @@
     </link>
     <joint name="camera_bottom_screw_frame_joint" type="fixed">
-        <origin xyz="0.01587 0.025 0.0125" rpy="0 0 0" />
-        <parent link="camera_bottom_screw_frame" />
-        <child link="camera_link" />
+        <origin xyz="-0.01587 -0.025 -0.0125" rpy="0 0 0" />
+        <parent link="camera_link" />
+        <child link="camera_bottom_screw_frame" />
         <axis xyz="0 0 0" />
     </joint>
@@ -303,11 +304,3 @@
         <axis xyz="0 0 0" />
     </joint>
-    <!-- Alla fine aggiungi il joint che collega il Gemini alla testa -->
-    <joint name="head_camera_joint" type="fixed">
-      <!-- usa gli offset che avevi nel tuo URDF per la camera finta -->
-      <origin xyz="0.062346 -0.000241 0.034324" rpy="0 0 0"/>
-      <parent link="${parent_link}"/>
-      <child link="camera_bottom_screw_frame"/>
-    </joint>
-  </xacro:macro>
 </robot>

File: urdf/materials.xacro (robot description, xacro)
@@ -2,5 +2,8 @@
 <robot name="rakuda" xmlns:xacro="http://www.ros.org/wiki/xacro" >
 <material name="silver">
-  <color rgba="0.700 0.700 0.700 1.000"/>
+  <color rgba="0.7 0.7 0.7 1.0"/>
+</material>
+<material name="white">
+  <color rgba="0.95 0.95 0.95 1.0"/>
 </material>
 </robot>

File: urdf/rakuda (copy).xacro (robot description, xacro)
@@ -111,5 +111,19 @@
   </collision>
 </link>
-<xacro:gemini_335_336 parent_link="neck_pitch_link" />
+<link name="head_camera_link">
+<!-- TODO: replace this mass and inertial with official Orbbec camera URDF values -->
+  <inertial>
+    <origin xyz="-0.0009302798678163388 -2.567747878634704e-07 0.0006112316563195441" rpy="0 0 0"/>
+    <mass value="0.00038890961357324327"/>
+    <inertia ixx="0" iyy="0" izz="0" ixy="0" iyz="0" ixz="0"/>
+  </inertial>
+  <visual>
+    <origin xyz="-0.062346 0.000141 -0.494924" rpy="0 0 0"/>
+    <geometry>
+      <mesh filename="file://$(find rakuda_description)/meshes/visual/head_camera_link.stl" scale="0.001 0.001 0.001"/>
+    </geometry>
+    <material name="white"/>
+  </visual>
+</link>
 <link name="l_link1">
   <inertial>
@@ -457,4 +471,9 @@
   <axis xyz="0.0 -1.0 0.0"/>
   <limit upper="0.610865" lower="-0.872665" effort="100" velocity="100"/>
+</joint>
+<joint name="head_camera_joint" type="fixed">
+  <origin xyz="0.062346 -0.000241 0.034324" rpy="0 0 0"/>
+  <parent link="neck_pitch_link"/>
+  <child link="head_camera_link"/>
 </joint>
 <joint name="l_arm_joint1" type="revolute">
