Commit message: tuning

File: urdf/camera_test.xacro (robot description, xacro)
@@ -58,5 +58,5 @@
 <!-- Joints -->
 <joint name="base_waist_joint" type="fixed">
-  <origin xyz="0.0 0.0 0.302" rpy="0 0 0"/>
+  <origin xyz="0.0 0.0 0.306" rpy="0 0 0"/>
   <parent link="base_link"/>
   <child link="waist_link"/>

File: urdf/rakuda.xacro (robot description, xacro)
@@ -432,5 +432,5 @@
 <!-- Joints -->
 <joint name="base_waist_joint" type="fixed">
-  <origin xyz="0.0 0.0 0.302" rpy="0 0 0"/>
+  <origin xyz="0.0 0.0 0.306" rpy="0 0 0"/>
   <parent link="base_link"/>
   <child link="waist_link"/>
