Commit message: renaming of links

File: urdf/rakuda.xacro (robot description, xacro)
@@ -20,5 +20,5 @@
     <origin xyz="0 0 0" rpy="0 0 0"/>
     <geometry>
-      <mesh filename="file://$(find rakuda_description)/meshes/collision/base_link.stl" scale="0.001 0.001 0.001"/>
+      <mesh filename="file://$(find rakuda_description)/meshes/collision/base_link_collision.stl" scale="0.001 0.001 0.001"/>
     </geometry>
   </collision>
@@ -40,9 +40,9 @@
     <origin xyz="0.0 0.0 -0.302" rpy="0 0 0"/>
     <geometry>
-      <mesh filename="file://$(find rakuda_description)/meshes/waist_link_1.stl" scale="0.001 0.001 0.001"/>
-    </geometry>
-  </collision>
-</link>
-<link name="torso_link_1">
+      <mesh filename="file://$(find rakuda_description)/meshes/collision/waist_link_collision.stl" scale="0.001 0.001 0.001"/>
+    </geometry>
+  </collision>
+</link>
+<link name="torso_link">
   <inertial>
     <origin xyz="-0.005791332469439025 1.1532258378440722e-08 0.06653504643352193" rpy="0 0 0"/>
@@ -53,5 +53,5 @@
     <origin xyz="-0.0 -0.0 -0.3085" rpy="0 0 0"/>
     <geometry>
-      <mesh filename="file://$(find rakuda_description)/meshes/torso_link_1.stl" scale="0.001 0.001 0.001"/>
+      <mesh filename="file://$(find rakuda_description)/meshes/torso_link_.stl" scale="0.001 0.001 0.001"/>
     </geometry>
     <material name="silver"/>
@@ -60,9 +60,9 @@
     <origin xyz="-0.0 -0.0 -0.3085" rpy="0 0 0"/>
     <geometry>
-      <mesh filename="file://$(find rakuda_description)/meshes/torso_link_1.stl" scale="0.001 0.001 0.001"/>
-    </geometry>
-  </collision>
-</link>
-<link name="neck_yaw_link_1">
+      <mesh filename="file://$(find rakuda_description)/meshes/collision/torso_link_collision.stl" scale="0.001 0.001 0.001"/>
+    </geometry>
+  </collision>
+</link>
+<link name="neck_yaw_link">
   <inertial>
     <origin xyz="2.8236692876973818e-15 -0.0003318177210791965 0.010126539608700469" rpy="0 0 0"/>
@@ -73,5 +73,5 @@
     <origin xyz="-0.0 -0.0 -0.43405" rpy="0 0 0"/>
     <geometry>
-      <mesh filename="file://$(find rakuda_description)/meshes/neck_yaw_link_1.stl" scale="0.001 0.001 0.001"/>
+      <mesh filename="file://$(find rakuda_description)/meshes/neck_yaw_link.stl" scale="0.001 0.001 0.001"/>
     </geometry>
     <material name="silver"/>
@@ -80,9 +80,9 @@
     <origin xyz="-0.0 -0.0 -0.43405" rpy="0 0 0"/>
     <geometry>
-      <mesh filename="file://$(find rakuda_description)/meshes/neck_yaw_link_1.stl" scale="0.001 0.001 0.001"/>
-    </geometry>
-  </collision>
-</link>
-<link name="neck_pitch_link_1">
+      <mesh filename="file://$(find rakuda_description)/meshes/collision/neck_yaw_link_collision.stl" scale="0.001 0.001 0.001"/>
+    </geometry>
+  </collision>
+</link>
+<link name="neck_pitch_link">
   <inertial>
     <origin xyz="0.008434802102082811 -0.0003276428199875459 0.04341435318306919" rpy="0 0 0"/>
@@ -93,5 +93,5 @@
     <origin xyz="0.0 -0.0001 -0.4606" rpy="0 0 0"/>
     <geometry>
-      <mesh filename="file://$(find rakuda_description)/meshes/neck_pitch_link_1.stl" scale="0.001 0.001 0.001"/>
+      <mesh filename="file://$(find rakuda_description)/meshes/neck_pitch_link.stl" scale="0.001 0.001 0.001"/>
     </geometry>
     <material name="silver"/>
@@ -100,9 +100,9 @@
     <origin xyz="0.0 -0.0001 -0.4606" rpy="0 0 0"/>
     <geometry>
-      <mesh filename="file://$(find rakuda_description)/meshes/neck_pitch_link_1.stl" scale="0.001 0.001 0.001"/>
-    </geometry>
-  </collision>
-</link>
-<link name="head_camera_link_1">
+      <mesh filename="file://$(find rakuda_description)/meshes/collision/neck_pitch_link_collision.stl" scale="0.001 0.001 0.001"/>
+    </geometry>
+  </collision>
+</link>
+<link name="head_camera_link">
   <inertial>
     <origin xyz="-0.0009302798678163388 -2.567747878634704e-07 0.0006112316563195441" rpy="0 0 0"/>
@@ -113,16 +113,10 @@
     <origin xyz="-0.062346 0.000141 -0.494924" rpy="0 0 0"/>
     <geometry>
-      <mesh filename="file://$(find rakuda_description)/meshes/head_camera_link_1.stl" scale="0.001 0.001 0.001"/>
-    </geometry>
-    <material name="silver"/>
-  </visual>
-  <collision>
-    <origin xyz="-0.062346 0.000141 -0.494924" rpy="0 0 0"/>
-    <geometry>
-      <mesh filename="file://$(find rakuda_description)/meshes/head_camera_link_1.stl" scale="0.001 0.001 0.001"/>
-    </geometry>
-  </collision>
-</link>
-<link name="l_link1_1">
+      <mesh filename="file://$(find rakuda_description)/meshes/head_camera_link.stl" scale="0.001 0.001 0.001"/>
+    </geometry>
+    <material name="silver"/>
+  </visual>
+</link>
+<link name="l_link1">
   <inertial>
     <origin xyz="8.165392508629886e-05 0.017114007906281148 -0.01682274344663298" rpy="0 0 0"/>
@@ -133,5 +127,5 @@
     <origin xyz="-0.0 -0.0826 -0.3946" rpy="0 0 0"/>
     <geometry>
-      <mesh filename="file://$(find rakuda_description)/meshes/l_link1_1.stl" scale="0.001 0.001 0.001"/>
+      <mesh filename="file://$(find rakuda_description)/meshes/l_link1.stl" scale="0.001 0.001 0.001"/>
     </geometry>
     <material name="silver"/>
@@ -140,9 +134,9 @@
     <origin xyz="-0.0 -0.0826 -0.3946" rpy="0 0 0"/>
     <geometry>
-      <mesh filename="file://$(find rakuda_description)/meshes/l_link1_1.stl" scale="0.001 0.001 0.001"/>
-    </geometry>
-  </collision>
-</link>
-<link name="r_link1_1">
+      <mesh filename="file://$(find rakuda_description)/meshes/collision/l_link1.stl" scale="0.001 0.001 0.001"/>
+    </geometry>
+  </collision>
+</link>
+<link name="r_link1">
   <inertial>
     <origin xyz="7.710992934052517e-05 -0.017114009124667 -0.016822741627550486" rpy="0 0 0"/>
@@ -153,5 +147,5 @@
     <origin xyz="-0.0 0.0826 -0.3946" rpy="0 0 0"/>
     <geometry>
-      <mesh filename="file://$(find rakuda_description)/meshes/r_link1_1.stl" scale="0.001 0.001 0.001"/>
+      <mesh filename="file://$(find rakuda_description)/meshes/r_link1.stl" scale="0.001 0.001 0.001"/>
     </geometry>
     <material name="silver"/>
@@ -160,9 +154,9 @@
     <origin xyz="-0.0 0.0826 -0.3946" rpy="0 0 0"/>
     <geometry>
-      <mesh filename="file://$(find rakuda_description)/meshes/r_link1_1.stl" scale="0.001 0.001 0.001"/>
-    </geometry>
-  </collision>
-</link>
-<link name="l_link2_1">
+      <mesh filename="file://$(find rakuda_description)/meshes/collision/r_link1_collision.stl" scale="0.001 0.001 0.001"/>
+    </geometry>
+  </collision>
+</link>
+<link name="l_link2">
   <inertial>
     <origin xyz="2.482738387163369e-05 0.000396191411047242 -0.03040144548272805" rpy="0 0 0"/>
@@ -173,5 +167,5 @@
     <origin xyz="-0.0 -0.1236 -0.3706" rpy="0 0 0"/>
     <geometry>
-      <mesh filename="file://$(find rakuda_description)/meshes/l_link2_1.stl" scale="0.001 0.001 0.001"/>
+      <mesh filename="file://$(find rakuda_description)/meshes/l_link2.stl" scale="0.001 0.001 0.001"/>
     </geometry>
     <material name="silver"/>
@@ -180,9 +174,9 @@
     <origin xyz="-0.0 -0.1236 -0.3706" rpy="0 0 0"/>
     <geometry>
-      <mesh filename="file://$(find rakuda_description)/meshes/l_link2_1.stl" scale="0.001 0.001 0.001"/>
-    </geometry>
-  </collision>
-</link>
-<link name="r_link2_1">
+      <mesh filename="file://$(find rakuda_description)/meshes/collision/l_link2_collision.stl" scale="0.001 0.001 0.001"/>
+    </geometry>
+  </collision>
+</link>
+<link name="r_link2">
   <inertial>
     <origin xyz="2.4825375508370262e-05 -0.0003961910521785711 -0.030401438771675282" rpy="0 0 0"/>
@@ -193,5 +187,5 @@
     <origin xyz="-0.0 0.1236 -0.3706" rpy="0 0 0"/>
     <geometry>
-      <mesh filename="file://$(find rakuda_description)/meshes/r_link2_1.stl" scale="0.001 0.001 0.001"/>
+      <mesh filename="file://$(find rakuda_description)/meshes/r_link2.stl" scale="0.001 0.001 0.001"/>
     </geometry>
     <material name="silver"/>
@@ -200,9 +194,9 @@
     <origin xyz="-0.0 0.1236 -0.3706" rpy="0 0 0"/>
     <geometry>
-      <mesh filename="file://$(find rakuda_description)/meshes/r_link2_1.stl" scale="0.001 0.001 0.001"/>
-    </geometry>
-  </collision>
-</link>
-<link name="l_link3_1">
+      <mesh filename="file://$(find rakuda_description)/meshes/collision/r_link2_collision.stl" scale="0.001 0.001 0.001"/>
+    </geometry>
+  </collision>
+</link>
+<link name="l_link3">
   <inertial>
     <origin xyz="0.012816931345662554 0.0004977011098152018 -0.019558162431457693" rpy="0 0 0"/>
@@ -213,5 +207,5 @@
     <origin xyz="-0.012 -0.1236 -0.2884" rpy="0 0 0"/>
     <geometry>
-      <mesh filename="file://$(find rakuda_description)/meshes/l_link3_1.stl" scale="0.001 0.001 0.001"/>
+      <mesh filename="file://$(find rakuda_description)/meshes/l_link3.stl" scale="0.001 0.001 0.001"/>
     </geometry>
     <material name="silver"/>
@@ -220,9 +214,9 @@
     <origin xyz="-0.012 -0.1236 -0.2884" rpy="0 0 0"/>
     <geometry>
-      <mesh filename="file://$(find rakuda_description)/meshes/l_link3_1.stl" scale="0.001 0.001 0.001"/>
-    </geometry>
-  </collision>
-</link>
-<link name="r_link3_1">
+      <mesh filename="file://$(find rakuda_description)/meshes/collision/l_link3_collision.stl" scale="0.001 0.001 0.001"/>
+    </geometry>
+  </collision>
+</link>
+<link name="r_link3">
   <inertial>
     <origin xyz="0.01281693134567282 -0.0004977011098376977 -0.019558162431519532" rpy="0 0 0"/>
@@ -233,5 +227,5 @@
     <origin xyz="-0.012 0.1236 -0.2884" rpy="0 0 0"/>
     <geometry>
-      <mesh filename="file://$(find rakuda_description)/meshes/r_link3_1.stl" scale="0.001 0.001 0.001"/>
+      <mesh filename="file://$(find rakuda_description)/meshes/r_link3.stl" scale="0.001 0.001 0.001"/>
     </geometry>
     <material name="silver"/>
@@ -240,9 +234,9 @@
     <origin xyz="-0.012 0.1236 -0.2884" rpy="0 0 0"/>
     <geometry>
-      <mesh filename="file://$(find rakuda_description)/meshes/r_link3_1.stl" scale="0.001 0.001 0.001"/>
-    </geometry>
-  </collision>
-</link>
-<link name="l_link4_1">
+      <mesh filename="file://$(find rakuda_description)/meshes/collision/r_link3_collision.stl" scale="0.001 0.001 0.001"/>
+    </geometry>
+  </collision>
+</link>
+<link name="l_link4">
   <inertial>
     <origin xyz="-0.013529205112779118 0.001169548907603693 -0.04421637055831898" rpy="0 0 0"/>
@@ -253,5 +247,5 @@
     <origin xyz="-0.036 -0.1236 -0.27035" rpy="0 0 0"/>
     <geometry>
-      <mesh filename="file://$(find rakuda_description)/meshes/l_link4_1.stl" scale="0.001 0.001 0.001"/>
+      <mesh filename="file://$(find rakuda_description)/meshes/l_link4.stl" scale="0.001 0.001 0.001"/>
     </geometry>
     <material name="silver"/>
@@ -260,9 +254,9 @@
     <origin xyz="-0.036 -0.1236 -0.27035" rpy="0 0 0"/>
     <geometry>
-      <mesh filename="file://$(find rakuda_description)/meshes/l_link4_1.stl" scale="0.001 0.001 0.001"/>
-    </geometry>
-  </collision>
-</link>
-<link name="r_link4_1">
+      <mesh filename="file://$(find rakuda_description)/meshes/collision/l_link4_collision.stl" scale="0.001 0.001 0.001"/>
+    </geometry>
+  </collision>
+</link>
+<link name="r_link4">
   <inertial>
     <origin xyz="-0.013529205589267821 -0.0011695493323802958 -0.04421637085671126" rpy="0 0 0"/>
@@ -273,5 +267,5 @@
     <origin xyz="-0.036 0.1236 -0.27035" rpy="0 0 0"/>
     <geometry>
-      <mesh filename="file://$(find rakuda_description)/meshes/r_link4_1.stl" scale="0.001 0.001 0.001"/>
+      <mesh filename="file://$(find rakuda_description)/meshes/r_link4.stl" scale="0.001 0.001 0.001"/>
     </geometry>
     <material name="silver"/>
@@ -280,9 +274,9 @@
     <origin xyz="-0.036 0.1236 -0.27035" rpy="0 0 0"/>
     <geometry>
-      <mesh filename="file://$(find rakuda_description)/meshes/r_link4_1.stl" scale="0.001 0.001 0.001"/>
-    </geometry>
-  </collision>
-</link>
-<link name="l_link5_1">
+      <mesh filename="file://$(find rakuda_description)/meshes/collision/r_link4_collision.stl" scale="0.001 0.001 0.001"/>
+    </geometry>
+  </collision>
+</link>
+<link name="l_link5">
   <inertial>
     <origin xyz="-0.00010745262237027431 0.0004983218880769968 -0.02809682280934908" rpy="0 0 0"/>
@@ -293,5 +287,5 @@
     <origin xyz="-0.036 -0.1236 -0.2049" rpy="0 0 0"/>
     <geometry>
-      <mesh filename="file://$(find rakuda_description)/meshes/l_link5_1.stl" scale="0.001 0.001 0.001"/>
+      <mesh filename="file://$(find rakuda_description)/meshes/l_link5.stl" scale="0.001 0.001 0.001"/>
     </geometry>
     <material name="silver"/>
@@ -300,9 +294,9 @@
     <origin xyz="-0.036 -0.1236 -0.2049" rpy="0 0 0"/>
     <geometry>
-      <mesh filename="file://$(find rakuda_description)/meshes/l_link5_1.stl" scale="0.001 0.001 0.001"/>
-    </geometry>
-  </collision>
-</link>
-<link name="r_link5_1">
+      <mesh filename="file://$(find rakuda_description)/meshes/collision/l_link5_collision.stl" scale="0.001 0.001 0.001"/>
+    </geometry>
+  </collision>
+</link>
+<link name="r_link5">
   <inertial>
     <origin xyz="-0.00010749374651377458 -0.00049827898943898 -0.02809678801928564" rpy="0 0 0"/>
@@ -313,5 +307,5 @@
     <origin xyz="-0.036 0.1236 -0.2049" rpy="0 0 0"/>
     <geometry>
-      <mesh filename="file://$(find rakuda_description)/meshes/r_link5_1.stl" scale="0.001 0.001 0.001"/>
+      <mesh filename="file://$(find rakuda_description)/meshes/r_link5.stl" scale="0.001 0.001 0.001"/>
     </geometry>
     <material name="silver"/>
@@ -320,9 +314,9 @@
     <origin xyz="-0.036 0.1236 -0.2049" rpy="0 0 0"/>
     <geometry>
-      <mesh filename="file://$(find rakuda_description)/meshes/r_link5_1.stl" scale="0.001 0.001 0.001"/>
-    </geometry>
-  </collision>
-</link>
-<link name="r_link6_1">
+      <mesh filename="file://$(find rakuda_description)/meshes/collision/r_link5.stl" scale="0.001 0.001 0.001"/>
+    </geometry>
+  </collision>
+</link>
+<link name="r_link6">
   <inertial>
     <origin xyz="0.0004978784895699889 -0.003188942119494928 -0.03994743914308038" rpy="0 0 0"/>
@@ -333,5 +327,5 @@
     <origin xyz="-0.036 0.1236 -0.16585" rpy="0 0 0"/>
     <geometry>
-      <mesh filename="file://$(find rakuda_description)/meshes/r_link6_1.stl" scale="0.001 0.001 0.001"/>
+      <mesh filename="file://$(find rakuda_description)/meshes/r_link6.stl" scale="0.001 0.001 0.001"/>
     </geometry>
     <material name="silver"/>
@@ -340,9 +334,9 @@
     <origin xyz="-0.036 0.1236 -0.16585" rpy="0 0 0"/>
     <geometry>
-      <mesh filename="file://$(find rakuda_description)/meshes/r_link6_1.stl" scale="0.001 0.001 0.001"/>
-    </geometry>
-  </collision>
-</link>
-<link name="l_link6_1">
+      <mesh filename="file://$(find rakuda_description)/meshes/collision/r_link6_collision.stl" scale="0.001 0.001 0.001"/>
+    </geometry>
+  </collision>
+</link>
+<link name="l_link6">
   <inertial>
     <origin xyz="0.000497878489597231 0.00318894211964936 -0.03994743914314852" rpy="0 0 0"/>
@@ -353,5 +347,5 @@
     <origin xyz="-0.036 -0.1236 -0.16585" rpy="0 0 0"/>
     <geometry>
-      <mesh filename="file://$(find rakuda_description)/meshes/l_link6_1.stl" scale="0.001 0.001 0.001"/>
+      <mesh filename="file://$(find rakuda_description)/meshes/l_link6.stl" scale="0.001 0.001 0.001"/>
     </geometry>
     <material name="silver"/>
@@ -360,9 +354,9 @@
     <origin xyz="-0.036 -0.1236 -0.16585" rpy="0 0 0"/>
     <geometry>
-      <mesh filename="file://$(find rakuda_description)/meshes/l_link6_1.stl" scale="0.001 0.001 0.001"/>
-    </geometry>
-  </collision>
-</link>
-<link name="r_gripper_a_1">
+      <mesh filename="file://$(find rakuda_description)/meshes/collision/l_link6_collision.stl" scale="0.001 0.001 0.001"/>
+    </geometry>
+  </collision>
+</link>
+<link name="r_gripper_a">
   <inertial>
     <origin xyz="-8.852479904033345e-05 -0.003089211052713342 -0.02999149965192692" rpy="0 0 0"/>
@@ -373,5 +367,5 @@
     <origin xyz="-0.036 0.1396 -0.1236" rpy="0 0 0"/>
     <geometry>
-      <mesh filename="file://$(find rakuda_description)/meshes/r_gripper_a_1.stl" scale="0.001 0.001 0.001"/>
+      <mesh filename="file://$(find rakuda_description)/meshes/r_gripper_a.stl" scale="0.001 0.001 0.001"/>
     </geometry>
     <material name="silver"/>
@@ -380,9 +374,9 @@
     <origin xyz="-0.036 0.1396 -0.1236" rpy="0 0 0"/>
     <geometry>
-      <mesh filename="file://$(find rakuda_description)/meshes/r_gripper_a_1.stl" scale="0.001 0.001 0.001"/>
-    </geometry>
-  </collision>
-</link>
-<link name="r_gripper_b_1">
+      <mesh filename="file://$(find rakuda_description)/meshes/collision/r_gripper_a_collision.stl" scale="0.001 0.001 0.001"/>
+    </geometry>
+  </collision>
+</link>
+<link name="r_gripper_b">
   <inertial>
     <origin xyz="-0.025089405701819327 0.003104658168288782 -0.030279426009768864" rpy="0 0 0"/>
@@ -393,5 +387,5 @@
     <origin xyz="-0.061 0.1156 -0.12355" rpy="0 0 0"/>
     <geometry>
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