Commit message: inertials to e06

File: urdf/rakuda.xacro (robot description, xacro)
@@ -8,5 +8,5 @@
     <origin xyz="-0.020408922979267937 -4.8555006463835264e-05 0.05284203414197219" rpy="0 0 0"/>
     <mass value="1.1379124037846244"/>
-    <inertia ixx="0.005787" iyy="0.006743" izz="0.003335" ixy="-4e-06" iyz="-2e-06" ixz="-0.000576"/>
+    <inertia ixx="5787e-06" iyy="6743e-06" izz="3335e-06" ixy="-4e-06" iyz="-2e-06" ixz="-576e-06"/>
   </inertial>
   <visual>
@@ -28,5 +28,5 @@
     <origin xyz="0.00015195021146941867 -2.820226960486473e-06 -0.004137928658236423" rpy="0 0 0"/>
     <mass value="0.04400005195575271"/>
-    <inertia ixx="1e-05" iyy="1.3e-05" izz="1.7e-05" ixy="-0.0" iyz="0.0" ixz="0.0"/>
+    <inertia ixx="10e-06" iyy="13e-06" izz="17e-06" ixy="0" iyz="0" ixz="0"/>
   </inertial>
   <visual>
@@ -48,5 +48,5 @@
     <origin xyz="-0.005791332469439025 1.1532258378440722e-08 0.06653504643352193" rpy="0 0 0"/>
     <mass value="0.7540141547961345"/>
-    <inertia ixx="0.001985" iyy="0.000909" izz="0.001513" ixy="0.0" iyz="0.0" ixz="-5.5e-05"/>
+    <inertia ixx="1985e-06" iyy="909e-06" izz="1513e-06" ixy="0" iyz="0" ixz="-55e-06"/>
   </inertial>
   <visual>
@@ -68,5 +68,5 @@
     <origin xyz="2.8236692876973818e-15 -0.0003318177210791965 0.010126539608700469" rpy="0 0 0"/>
     <mass value="0.01399997346170466"/>
-    <inertia ixx="5e-06" iyy="3e-06" izz="4e-06" ixy="0.0" iyz="0.0" ixz="-0.0"/>
+    <inertia ixx="5e-06" iyy="3e-06" izz="4e-06" ixy="0" iyz="0" ixz="0"/>
   </inertial>
   <visual>
@@ -88,5 +88,5 @@
     <origin xyz="0.008434802102082811 -0.0003276428199875459 0.04341435318306919" rpy="0 0 0"/>
     <mass value="0.2822100615108845"/>
-    <inertia ixx="0.000695" iyy="0.000648" izz="0.000763" ixy="-0.0" iyz="-1e-06" ixz="4.2e-05"/>
+    <inertia ixx="695e-06" iyy="648e-06" izz="763e-06" ixy="0" iyz="-1e-06" ixz="42e-06"/>
   </inertial>
   <visual>
@@ -105,8 +105,9 @@
 </link>
 <link name="head_camera_link">
+<!-- TODO: replace this mass and inertial with official Orbbec camera URDF values -->
   <inertial>
     <origin xyz="-0.0009302798678163388 -2.567747878634704e-07 0.0006112316563195441" rpy="0 0 0"/>
     <mass value="0.00038890961357324327"/>
-    <inertia ixx="0.0" iyy="0.0" izz="0.0" ixy="-0.0" iyz="-0.0" ixz="-0.0"/>
+    <inertia ixx="0" iyy="0" izz="0" ixy="0" iyz="0" ixz="0"/>
   </inertial>
   <visual>
@@ -122,5 +123,5 @@
     <origin xyz="8.165392508629886e-05 0.017114007906281148 -0.01682274344663298" rpy="0 0 0"/>
     <mass value="0.07299177430140238"/>
-    <inertia ixx="4e-05" iyy="5.1e-05" izz="5.7e-05" ixy="-0.0" iyz="8e-06" ixz="0.0"/>
+    <inertia ixx="40e-06" iyy="51e-06" izz="57e-06" ixy="0" iyz="8e-06" ixz="0"/>
   </inertial>
   <visual>
@@ -142,5 +143,5 @@
     <origin xyz="7.710992934052517e-05 -0.017114009124667 -0.016822741627550486" rpy="0 0 0"/>
     <mass value="0.07299176592385347"/>
-    <inertia ixx="4e-05" iyy="5.1e-05" izz="5.7e-05" ixy="0.0" iyz="-8e-06" ixz="0.0"/>
+    <inertia ixx="40e-06" iyy="51e-06" izz="57e-06" ixy="0" iyz="-8e-06" ixz="0"/>
   </inertial>
   <visual>
@@ -162,5 +163,5 @@
     <origin xyz="2.482738387163369e-05 0.000396191411047242 -0.03040144548272805" rpy="0 0 0"/>
     <mass value="0.2900252815965671"/>
-    <inertia ixx="0.000279" iyy="0.000303" izz="0.000102" ixy="-1e-06" iyz="-2e-06" ixz="-7e-06"/>
+    <inertia ixx="279e-06" iyy="303e-06" izz="102e-06" ixy="-1e-06" iyz="-2e-06" ixz="-7e-06"/>
   </inertial>
   <visual>
@@ -202,5 +203,5 @@
     <origin xyz="0.012816931345662554 0.0004977011098152018 -0.019558162431457693" rpy="0 0 0"/>
     <mass value="0.10799652996016351"/>
-    <inertia ixx="2.5e-05" iyy="4.3e-05" izz="4e-05" ixy="-0.0" iyz="-0.0" ixz="1e-06"/>
+    <inertia ixx="25e-06" iyy="43e-06" izz="40e-06" ixy="0" iyz="0" ixz="1e-06"/>
   </inertial>
   <visual>
@@ -222,5 +223,5 @@
     <origin xyz="0.01281693134567282 -0.0004977011098376977 -0.019558162431519532" rpy="0 0 0"/>
     <mass value="0.10799652996026934"/>
-    <inertia ixx="2.5e-05" iyy="4.3e-05" izz="4e-05" ixy="0.0" iyz="0.0" ixz="1e-06"/>
+    <inertia ixx="25e-06" iyy="43e-06" izz="40e-06" ixy="0" iyz="0" ixz="1e-06"/>
   </inertial>
   <visual>
@@ -242,5 +243,5 @@
     <origin xyz="-0.013529205112779118 0.001169548907603693 -0.04421637055831898" rpy="0 0 0"/>
     <mass value="0.10699509679197633"/>
-    <inertia ixx="3e-05" iyy="4.3e-05" izz="3.6e-05" ixy="1e-06" iyz="0.0" ixz="-2e-06"/>
+    <inertia ixx="30e-06" iyy="43e-06" izz="36e-06" ixy="1e-06" iyz="0" ixz="-2e-06"/>
   </inertial>
   <visual>
@@ -262,5 +263,5 @@
     <origin xyz="-0.013529205589267821 -0.0011695493323802958 -0.04421637085671126" rpy="0 0 0"/>
     <mass value="0.10699509934326328"/>
-    <inertia ixx="3e-05" iyy="4.3e-05" izz="3.6e-05" ixy="-1e-06" iyz="-0.0" ixz="-2e-06"/>
+    <inertia ixx="30e-06" iyy="43e-06" izz="36e-06" ixy="-1e-06" iyz="0" ixz="-2e-06"/>
   </inertial>
   <visual>
@@ -282,5 +283,5 @@
     <origin xyz="-0.00010745262237027431 0.0004983218880769968 -0.02809682280934908" rpy="0 0 0"/>
     <mass value="0.10899653712889695"/>
-    <inertia ixx="4e-05" iyy="4.4e-05" izz="2.6e-05" ixy="-0.0" iyz="0.0" ixz="0.0"/>
+    <inertia ixx="40e-06" iyy="44e-06" izz="26e-06" ixy="0" iyz="0" ixz="0"/>
   </inertial>
   <visual>
@@ -302,5 +303,5 @@
     <origin xyz="-0.00010749374651377458 -0.00049827898943898 -0.02809678801928564" rpy="0 0 0"/>
     <mass value="0.10899673027569862"/>
-    <inertia ixx="4e-05" iyy="4.4e-05" izz="2.6e-05" ixy="0.0" iyz="-0.0" ixz="0.0"/>
+    <inertia ixx="40e-06" iyy="44e-06" izz="26e-06" ixy="0" iyz="0" ixz="0"/>
   </inertial>
   <visual>
@@ -322,5 +323,5 @@
     <origin xyz="0.0004978784895699889 -0.003188942119494928 -0.03994743914308038" rpy="0 0 0"/>
     <mass value="0.07399870180333049"/>
-    <inertia ixx="2.3e-05" iyy="1.7e-05" izz="2.2e-05" ixy="0.0" iyz="-0.0" ixz="0.0"/>
+    <inertia ixx="23e-06" iyy="17e-06" izz="22e-06" ixy="0" iyz="0" ixz="0"/>
   </inertial>
   <visual>
@@ -342,5 +343,5 @@
     <origin xyz="0.000497878489597231 0.00318894211964936 -0.03994743914314852" rpy="0 0 0"/>
     <mass value="0.07399870180299768"/>
-    <inertia ixx="2.3e-05" iyy="1.7e-05" izz="2.2e-05" ixy="-0.0" iyz="0.0" ixz="0.0"/>
+    <inertia ixx="23e-06" iyy="17e-06" izz="22e-06" ixy="0" iyz="0" ixz="0"/>
   </inertial>
   <visual>
@@ -362,5 +363,5 @@
     <origin xyz="-8.852479904033345e-05 -0.003089211052713342 -0.02999149965192692" rpy="0 0 0"/>
     <mass value="0.017998423512260126"/>
-    <inertia ixx="6e-06" iyy="1e-05" izz="5e-06" ixy="0.0" iyz="0.0" ixz="-0.0"/>
+    <inertia ixx="6e-06" iyy="10e-06" izz="5e-06" ixy="0" iyz="0" ixz="0"/>
   </inertial>
   <visual>
@@ -382,5 +383,5 @@
     <origin xyz="-0.025089405701819327 0.003104658168288782 -0.030279426009768864" rpy="0 0 0"/>
     <mass value="0.018999892317782645"/>
-    <inertia ixx="6e-06" iyy="1e-05" izz="5e-06" ixy="-0.0" iyz="-0.0" ixz="-0.0"/>
+    <inertia ixx="6e-06" iyy="10e-06" izz="5e-06" ixy="0" iyz="0" ixz="0"/>
   </inertial>
   <visual>
@@ -402,5 +403,5 @@
     <origin xyz="-8.920360655783471e-05 0.003089714518583392 -0.029990508331487045" rpy="0 0 0"/>
     <mass value="0.017997801931831644"/>
-    <inertia ixx="6e-06" iyy="1e-05" izz="5e-06" ixy="-0.0" iyz="-0.0" ixz="-0.0"/>
+    <inertia ixx="6e-06" iyy="10e-06" izz="5e-06" ixy="0" iyz="0" ixz="0"/>
   </inertial>
   <visual>
@@ -422,5 +423,5 @@
     <origin xyz="-0.02508868291206493 -0.0031035251440137968 -0.030280490115251982" rpy="0 0 0"/>
     <mass value="0.019000550359800868"/>
-    <inertia ixx="6e-06" iyy="1e-05" izz="5e-06" ixy="0.0" iyz="0.0" ixz="-0.0"/>
+    <inertia ixx="6e-06" iyy="10e-06" izz="5e-06" ixy="0" iyz="0" ixz="0"/>
   </inertial>
   <visual>
@@ -457,5 +458,5 @@
   <limit upper="1.22173" lower="-1.22173" effort="100" velocity="100"/>
 </joint>
-<joint name="neck_pitch_join" type="revolute">
+<joint name="neck_pitch_joint" type="revolute">
   <origin xyz="-0.0 0.0001 0.02655" rpy="0 0 0"/>
   <parent link="neck_yaw_link"/>

Commit message: meshes in directories

File: urdf/rakuda.xacro (robot description, xacro)
@@ -33,5 +33,5 @@
     <origin xyz="0.0 0.0 -0.302" rpy="0 0 0"/>
     <geometry>
-      <mesh filename="file://$(find rakuda_description)/meshes/waist_link.stl" scale="0.001 0.001 0.001"/>
+      <mesh filename="file://$(find rakuda_description)/meshes/visual/waist_link.stl" scale="0.001 0.001 0.001"/>
     </geometry>
     <material name="silver"/>
@@ -53,5 +53,5 @@
     <origin xyz="-0.0 -0.0 -0.3085" rpy="0 0 0"/>
     <geometry>
-      <mesh filename="file://$(find rakuda_description)/meshes/torso_link_.stl" scale="0.001 0.001 0.001"/>
+      <mesh filename="file://$(find rakuda_description)/meshes/visual/torso_link_.stl" scale="0.001 0.001 0.001"/>
     </geometry>
     <material name="silver"/>
@@ -73,5 +73,5 @@
     <origin xyz="-0.0 -0.0 -0.43405" rpy="0 0 0"/>
     <geometry>
-      <mesh filename="file://$(find rakuda_description)/meshes/neck_yaw_link.stl" scale="0.001 0.001 0.001"/>
+      <mesh filename="file://$(find rakuda_description)/meshes/visual/neck_yaw_link.stl" scale="0.001 0.001 0.001"/>
     </geometry>
     <material name="silver"/>
@@ -93,5 +93,5 @@
     <origin xyz="0.0 -0.0001 -0.4606" rpy="0 0 0"/>
     <geometry>
-      <mesh filename="file://$(find rakuda_description)/meshes/neck_pitch_link.stl" scale="0.001 0.001 0.001"/>
+      <mesh filename="file://$(find rakuda_description)/meshes/visual/neck_pitch_link.stl" scale="0.001 0.001 0.001"/>
     </geometry>
     <material name="silver"/>
@@ -114,5 +114,5 @@
     <origin xyz="-0.062346 0.000141 -0.494924" rpy="0 0 0"/>
     <geometry>
-      <mesh filename="file://$(find rakuda_description)/meshes/head_camera_link.stl" scale="0.001 0.001 0.001"/>
+      <mesh filename="file://$(find rakuda_description)/meshes/visual/head_camera_link.stl" scale="0.001 0.001 0.001"/>
     </geometry>
     <material name="silver"/>
@@ -128,5 +128,5 @@
     <origin xyz="-0.0 -0.0826 -0.3946" rpy="0 0 0"/>
     <geometry>
-      <mesh filename="file://$(find rakuda_description)/meshes/l_link1.stl" scale="0.001 0.001 0.001"/>
+      <mesh filename="file://$(find rakuda_description)/meshes/visual/l_link1.stl" scale="0.001 0.001 0.001"/>
     </geometry>
     <material name="silver"/>
@@ -148,5 +148,5 @@
     <origin xyz="-0.0 0.0826 -0.3946" rpy="0 0 0"/>
     <geometry>
-      <mesh filename="file://$(find rakuda_description)/meshes/r_link1.stl" scale="0.001 0.001 0.001"/>
+      <mesh filename="file://$(find rakuda_description)/meshes/visual/r_link1.stl" scale="0.001 0.001 0.001"/>
     </geometry>
     <material name="silver"/>
@@ -168,5 +168,5 @@
     <origin xyz="-0.0 -0.1236 -0.3706" rpy="0 0 0"/>
     <geometry>
-      <mesh filename="file://$(find rakuda_description)/meshes/l_link2.stl" scale="0.001 0.001 0.001"/>
+      <mesh filename="file://$(find rakuda_description)/meshes/visual/l_link2.stl" scale="0.001 0.001 0.001"/>
     </geometry>
     <material name="silver"/>
@@ -188,5 +188,5 @@
     <origin xyz="-0.0 0.1236 -0.3706" rpy="0 0 0"/>
     <geometry>
-      <mesh filename="file://$(find rakuda_description)/meshes/r_link2.stl" scale="0.001 0.001 0.001"/>
+      <mesh filename="file://$(find rakuda_description)/meshes/visual/r_link2.stl" scale="0.001 0.001 0.001"/>
     </geometry>
     <material name="silver"/>
@@ -208,5 +208,5 @@
     <origin xyz="-0.012 -0.1236 -0.2884" rpy="0 0 0"/>
     <geometry>
-      <mesh filename="file://$(find rakuda_description)/meshes/l_link3.stl" scale="0.001 0.001 0.001"/>
+      <mesh filename="file://$(find rakuda_description)/meshes/visual/l_link3.stl" scale="0.001 0.001 0.001"/>
     </geometry>
     <material name="silver"/>
@@ -228,5 +228,5 @@
     <origin xyz="-0.012 0.1236 -0.2884" rpy="0 0 0"/>
     <geometry>
-      <mesh filename="file://$(find rakuda_description)/meshes/r_link3.stl" scale="0.001 0.001 0.001"/>
+      <mesh filename="file://$(find rakuda_description)/meshes/visual/r_link3.stl" scale="0.001 0.001 0.001"/>
     </geometry>
     <material name="silver"/>
@@ -248,5 +248,5 @@
     <origin xyz="-0.036 -0.1236 -0.27035" rpy="0 0 0"/>
     <geometry>
-      <mesh filename="file://$(find rakuda_description)/meshes/l_link4.stl" scale="0.001 0.001 0.001"/>
+      <mesh filename="file://$(find rakuda_description)/meshes/visual/l_link4.stl" scale="0.001 0.001 0.001"/>
     </geometry>
     <material name="silver"/>
@@ -268,5 +268,5 @@
     <origin xyz="-0.036 0.1236 -0.27035" rpy="0 0 0"/>
     <geometry>
-      <mesh filename="file://$(find rakuda_description)/meshes/r_link4.stl" scale="0.001 0.001 0.001"/>
+      <mesh filename="file://$(find rakuda_description)/meshes/visual/r_link4.stl" scale="0.001 0.001 0.001"/>
     </geometry>
     <material name="silver"/>
@@ -288,5 +288,5 @@
     <origin xyz="-0.036 -0.1236 -0.2049" rpy="0 0 0"/>
     <geometry>
-      <mesh filename="file://$(find rakuda_description)/meshes/l_link5.stl" scale="0.001 0.001 0.001"/>
+      <mesh filename="file://$(find rakuda_description)/meshes/visual/l_link5.stl" scale="0.001 0.001 0.001"/>
     </geometry>
     <material name="silver"/>
@@ -308,5 +308,5 @@
     <origin xyz="-0.036 0.1236 -0.2049" rpy="0 0 0"/>
     <geometry>
-      <mesh filename="file://$(find rakuda_description)/meshes/r_link5.stl" scale="0.001 0.001 0.001"/>
+      <mesh filename="file://$(find rakuda_description)/meshes/visual/r_link5.stl" scale="0.001 0.001 0.001"/>
     </geometry>
     <material name="silver"/>
@@ -328,5 +328,5 @@
     <origin xyz="-0.036 0.1236 -0.16585" rpy="0 0 0"/>
     <geometry>
-      <mesh filename="file://$(find rakuda_description)/meshes/r_link6.stl" scale="0.001 0.001 0.001"/>
+      <mesh filename="file://$(find rakuda_description)/meshes/visual/r_link6.stl" scale="0.001 0.001 0.001"/>
     </geometry>
     <material name="silver"/>
@@ -348,5 +348,5 @@
     <origin xyz="-0.036 -0.1236 -0.16585" rpy="0 0 0"/>
     <geometry>
-      <mesh filename="file://$(find rakuda_description)/meshes/l_link6.stl" scale="0.001 0.001 0.001"/>
+      <mesh filename="file://$(find rakuda_description)/meshes/visual/l_link6.stl" scale="0.001 0.001 0.001"/>
     </geometry>
     <material name="silver"/>
@@ -368,5 +368,5 @@
     <origin xyz="-0.036 0.1396 -0.1236" rpy="0 0 0"/>
     <geometry>
-      <mesh filename="file://$(find rakuda_description)/meshes/r_gripper_a.stl" scale="0.001 0.001 0.001"/>
+      <mesh filename="file://$(find rakuda_description)/meshes/visual/r_gripper_a.stl" scale="0.001 0.001 0.001"/>
     </geometry>
     <material name="silver"/>
@@ -388,5 +388,5 @@
     <origin xyz="-0.061 0.1156 -0.12355" rpy="0 0 0"/>
     <geometry>
-      <mesh filename="file://$(find rakuda_description)/meshes/r_gripper_b.stl" scale="0.001 0.001 0.001"/>
+      <mesh filename="file://$(find rakuda_description)/meshes/visual/r_gripper_b.stl" scale="0.001 0.001 0.001"/>
     </geometry>
     <material name="silver"/>
@@ -408,5 +408,5 @@
     <origin xyz="-0.036 -0.1396 -0.1236" rpy="0 0 0"/>
     <geometry>
-      <mesh filename="file://$(find rakuda_description)/meshes/l_gripper_a.stl" scale="0.001 0.001 0.001"/>
+      <mesh filename="file://$(find rakuda_description)/meshes/visual/l_gripper_a.stl" scale="0.001 0.001 0.001"/>
     </geometry>
     <material name="silver"/>
@@ -428,5 +428,5 @@
     <origin xyz="-0.061 -0.1156 -0.12355" rpy="0 0 0"/>
     <geometry>
-      <mesh filename="file://$(find rakuda_description)/meshes/l_gripper_b.stl" scale="0.001 0.001 0.001"/>
+      <mesh filename="file://$(find rakuda_description)/meshes/visual/l_gripper_b.stl" scale="0.001 0.001 0.001"/>
     </geometry>
     <material name="silver"/>

Commit message: Mimic joints

File: urdf/rakuda.xacro (robot description, xacro)
@@ -565,6 +565,6 @@
   <parent link="r_link6"/>
   <child link="r_gripper_b"/>
-  <axis xyz="1.0 -4.8e-05 -0.0"/>
-  <limit upper="1.22173" lower="0.0" effort="100" velocity="100"/>
+  <axis xyz="1.0 0.0 0.0"/>
+  <mimic joint="r_gripper_joint" multiplier="-1.0" offset="0.0"/>
 </joint>
 <joint name="l_gripper_joint" type="revolute">
@@ -579,6 +579,6 @@
   <parent link="l_link6"/>
   <child link="l_gripper_b"/>
-  <axis xyz="1.0 4.8e-05 -0.0"/>
-  <limit upper="0.0" lower="-1.22173" effort="100" velocity="100"/>
+  <axis xyz="1.0 0.0 0.0"/>
+  <mimic joint="l_gripper_joint" multiplier="-1.0" offset="0.0"/>
 </joint>
 </robot>

Commit message: bugfixses

File: urdf/rakuda.xacro (robot description, xacro)
@@ -53,5 +53,5 @@
     <origin xyz="-0.0 -0.0 -0.3085" rpy="0 0 0"/>
     <geometry>
-      <mesh filename="file://$(find rakuda_description)/meshes/visual/torso_link_.stl" scale="0.001 0.001 0.001"/>
+      <mesh filename="file://$(find rakuda_description)/meshes/visual/torso_link.stl" scale="0.001 0.001 0.001"/>
     </geometry>
     <material name="silver"/>
@@ -98,5 +98,5 @@
   </visual>
   <collision>
-    <origin xyz="0.0 -0.0001 -0.4606" rpy="0 0 0"/>
+    <origin xyz="0.5 -0.0001 -0.4606" rpy="0 0 0"/>
     <geometry>
       <mesh filename="file://$(find rakuda_description)/meshes/collision/neck_pitch_link_collision.stl" scale="0.001 0.001 0.001"/>
@@ -135,5 +135,5 @@
     <origin xyz="-0.0 -0.0826 -0.3946" rpy="0 0 0"/>
     <geometry>
-      <mesh filename="file://$(find rakuda_description)/meshes/collision/l_link1.stl" scale="0.001 0.001 0.001"/>
+      <mesh filename="file://$(find rakuda_description)/meshes/collision/l_link1_collision.stl" scale="0.001 0.001 0.001"/>
     </geometry>
   </collision>
@@ -315,5 +315,5 @@
     <origin xyz="-0.036 0.1236 -0.2049" rpy="0 0 0"/>
     <geometry>
-      <mesh filename="file://$(find rakuda_description)/meshes/collision/r_link5.stl" scale="0.001 0.001 0.001"/>
+      <mesh filename="file://$(find rakuda_description)/meshes/collision/r_link5_collision.stl" scale="0.001 0.001 0.001"/>
     </geometry>
   </collision>
@@ -415,5 +415,5 @@
     <origin xyz="-0.036 -0.1396 -0.1236" rpy="0 0 0"/>
     <geometry>
-      <mesh filename="file://$(find rakuda_description)/meshes/collision/l_gripper_a.stl" scale="0.001 0.001 0.001"/>
+      <mesh filename="file://$(find rakuda_description)/meshes/collision/l_gripper_a_collision.stl" scale="0.001 0.001 0.001"/>
     </geometry>
   </collision>
@@ -435,5 +435,5 @@
     <origin xyz="-0.061 -0.1156 -0.12355" rpy="0 0 0"/>
     <geometry>
-      <mesh filename="file://$(find rakuda_description)/meshes/collision/l_gripper_b.stl" scale="0.001 0.001 0.001"/>
+      <mesh filename="file://$(find rakuda_description)/meshes/collision/l_gripper_b_collision.stl" scale="0.001 0.001 0.001"/>
     </geometry>
   </collision>
@@ -563,4 +563,5 @@
 <joint name="r_gripper_mimic_joint" type="revolute">
   <origin xyz="0.025 0.008 -0.0423" rpy="0 0 0"/>
+  <limit lower="-1.0" upper="0.01" effort="10" velocity="1.0"/>
   <parent link="r_link6"/>
   <child link="r_gripper_b"/>
@@ -577,4 +578,5 @@
 <joint name="l_gripper_mimic_joint" type="revolute">
   <origin xyz="0.025 -0.008 -0.0423" rpy="0 0 0"/>
+  <limit lower="-0.01" upper="1.0" effort="10" velocity="1.0"/>
   <parent link="l_link6"/>
   <child link="l_gripper_b"/>

Commit message: Fix on intertial

File: urdf/rakuda.xacro (robot description, xacro)
@@ -381,10 +381,10 @@
 <link name="r_gripper_b">
   <inertial>
-    <origin xyz="-0.025089405701819327 0.003104658168288782 -0.030279426009768864" rpy="0 0 0"/>
+    <origin xyz="-8.852479904033345e-05 0.003104658168288782 -0.030279426009768864" rpy="0 0 0"/>
     <mass value="0.018999892317782645"/>
     <inertia ixx="6e-06" iyy="10e-06" izz="5e-06" ixy="0" iyz="0" ixz="0"/>
   </inertial>
   <visual>
-    <origin xyz="-0.061 0.1156 -0.12355" rpy="0 0 0"/>
+    <origin xyz="-0.036 0.1156 -0.12355" rpy="0 0 0"/>
     <geometry>
       <mesh filename="file://$(find rakuda_description)/meshes/visual/r_gripper_b.stl" scale="0.001 0.001 0.001"/>
@@ -393,5 +393,5 @@
   </visual>
   <collision>
-    <origin xyz="-0.061 0.1156 -0.12355" rpy="0 0 0"/>
+    <origin xyz="-0.036 0.1156 -0.12355" rpy="0 0 0"/>
     <geometry>
       <mesh filename="file://$(find rakuda_description)/meshes/collision/r_gripper_b_collision.stl" scale="0.001 0.001 0.001"/>
@@ -421,10 +421,10 @@
 <link name="l_gripper_b">
   <inertial>
-    <origin xyz="-0.02508868291206493 -0.0031035251440137968 -0.030280490115251982" rpy="0 0 0"/>
+    <origin xyz="-8.920360655783471e-05 -0.0031035251440137968 -0.030280490115251982" rpy="0 0 0"/>
     <mass value="0.019000550359800868"/>
     <inertia ixx="6e-06" iyy="10e-06" izz="5e-06" ixy="0" iyz="0" ixz="0"/>
   </inertial>
   <visual>
-    <origin xyz="-0.061 -0.1156 -0.12355" rpy="0 0 0"/>
+    <origin xyz="-0.036 -0.1156 -0.12355" rpy="0 0 0"/>
     <geometry>
       <mesh filename="file://$(find rakuda_description)/meshes/visual/l_gripper_b.stl" scale="0.001 0.001 0.001"/>
@@ -433,5 +433,5 @@
   </visual>
   <collision>
-    <origin xyz="-0.061 -0.1156 -0.12355" rpy="0 0 0"/>
+    <origin xyz="-0.036 -0.1156 -0.12355" rpy="0 0 0"/>
     <geometry>
       <mesh filename="file://$(find rakuda_description)/meshes/collision/l_gripper_b_collision.stl" scale="0.001 0.001 0.001"/>
@@ -562,5 +562,5 @@
 </joint>
 <joint name="r_gripper_mimic_joint" type="revolute">
-  <origin xyz="0.025 0.008 -0.0423" rpy="0 0 0"/>
+  <origin xyz="0.0 0.008 -0.0423" rpy="0 0 0"/>
   <limit lower="-1.0" upper="0.01" effort="10" velocity="1.0"/>
   <parent link="r_link6"/>
@@ -577,5 +577,5 @@
 </joint>
 <joint name="l_gripper_mimic_joint" type="revolute">
-  <origin xyz="0.025 -0.008 -0.0423" rpy="0 0 0"/>
+  <origin xyz="0.0 -0.008 -0.0423" rpy="0 0 0"/>
   <limit lower="-0.01" upper="1.0" effort="10" velocity="1.0"/>
   <parent link="l_link6"/>
