Commit message: dummy link for base_link inertial

File: urdf/rakuda.xacro (robot description, xacro)
@@ -27,4 +27,19 @@
 <!-- Main links -->
 <link name="base_link">
+  <visual>
+    <origin xyz="0 0 0" rpy="0 0 0"/>
+    <geometry>
+      <mesh filename="file://$(find rakuda_description)/meshes/visual/base_link.stl" scale="0.001 0.001 0.001"/>
+    </geometry>
+    <material name="white"/>
+  </visual>
+  <collision>
+    <origin xyz="0 0 0" rpy="0 0 0"/>
+    <geometry>
+      <mesh filename="file://$(find rakuda_description)/meshes/collision/base_link_collision.stl" scale="0.001 0.001 0.001"/>
+    </geometry>
+  </collision>
+</link>
+<link name="base_inertia_link">
   <inertial>
     <origin xyz="-0.020408922979267937 -4.8555006463835264e-05 0.05284203414197219" rpy="0 0 0"/>
@@ -32,18 +47,10 @@
     <inertia ixx="5787e-06" iyy="6743e-06" izz="3335e-06" ixy="-4e-06" iyz="-2e-06" ixz="-576e-06"/>
   </inertial>
-  <visual>
-    <origin xyz="0 0 0" rpy="0 0 0"/>
-    <geometry>
-      <mesh filename="file://$(find rakuda_description)/meshes/visual/base_link.stl" scale="0.001 0.001 0.001"/>
-    </geometry>
-    <material name="white"/>
-  </visual>
-  <collision>
-    <origin xyz="0 0 0" rpy="0 0 0"/>
-    <geometry>
-      <mesh filename="file://$(find rakuda_description)/meshes/collision/base_link_collision.stl" scale="0.001 0.001 0.001"/>
-    </geometry>
-  </collision>
-</link>
+</link>
+<joint name="base_inertia_joint" type="fixed">
+  <parent link="base_link"/>
+  <child link="base_inertia_link"/>
+  <origin xyz="0 0 0" rpy="0 0 0"/>
+</joint>
 <link name="waist_link">
   <inertial>
