Commit message: bugfix

File: urdf/gemini_335_336.urdf.xacro (robot description, xacro)
@@ -3,5 +3,5 @@
   <!-- proprietà per i mesh -->
   <xacro:property name="mesh_path" value="package://orbbec_description/meshes/gemini335_336/" />
-  <!-- macro che istanzia il Gemini e lo attacca a un parent -->
+  <!-- macro che istanzia la Orbbec e la attacca al parent -->
   <xacro:macro name="gemini_335_336" params="parent_link">
     <link name="camera_link">
@@ -14,5 +14,5 @@
         </inertial>
         <visual>
-            <origin xyz="-0.01587 -0.025 -0.0125" rpy="0 0 0" />
+            <origin xyz="0 0 0" rpy="0 0 0" />
             <geometry>
                 <mesh filename="${mesh_path}camera_link.STL" />
@@ -54,7 +54,7 @@
     </link>
     <joint name="camera_bottom_screw_frame_joint" type="fixed">
-        <origin xyz="0.01587 0.025 0.0125" rpy="0 0 0" />
-        <parent link="camera_bottom_screw_frame" />
-        <child link="camera_link" />
+        <origin xyz="0 0 0" rpy="0 0 0" />
+        <parent link="camera_link" />
+        <child link="camera_bottom_screw_frame" />
         <axis xyz="0 0 0" />
     </joint>
@@ -85,6 +85,6 @@
     </link>
     <joint name="camera_left_ir_joint" type="fixed">
-        <origin xyz="0 0 0" rpy="0 0 0" />
-        <parent link="camera_depth_frame" />
+        <origin xyz="0.01587 -0.025 0.0125" rpy="0 0 0" />
+        <parent link="camera_bottom_screw_frame" />
         <child link="camera_left_ir_frame" />
         <axis xyz="0 0 0" />
@@ -115,6 +115,6 @@
     </link>
     <joint name="camera_left_ir_optical_joint" type="fixed">
-        <origin xyz="0 0 0" rpy="-1.5707963267949 0 -1.5707963267949" />
-        <parent link="camera_left_ir_frame" />
+        <origin xyz="0.01587 -0.025 0.0125" rpy="-1.5707963267949 0 -1.5707963267949" />
+        <parent link="camera_bottom_screw_frame" />
         <child link="camera_left_ir_optical_frame" />
         <axis xyz="0 0 0" />
@@ -146,6 +146,6 @@
     </link>
     <joint name="camera_right_ir_joint" type="fixed">
-        <origin xyz="0 -0.05 0" rpy="0 0 0" />
-        <parent link="camera_depth_frame" />
+        <origin xyz="0.01587 0.025 0.0125" rpy="0 0 0" />
+        <parent link="camera_bottom_screw_frame" />
         <child link="camera_right_ir_frame" />
         <axis xyz="0 0 0" />
@@ -176,6 +176,6 @@
     </link>
     <joint name="camera_right_ir_optical_joint" type="fixed">
-        <origin xyz="0 0 0" rpy="-1.5707963267949 0 -1.5707963267949" />
-        <parent link="camera_right_ir_frame" />
+        <origin xyz="0.01587 0.025 0.0125" rpy="-1.5707963267949 0 -1.5707963267949" />
+        <parent link="camera_bottom_screw_frame" />
         <child link="camera_right_ir_optical_frame" />
         <axis xyz="0 0 0" />
@@ -207,6 +207,6 @@
     </link>
     <joint name="camera_color_joint" type="fixed">
-        <origin xyz="0.001663 -0.014005 0.000005" rpy="0 0 0" />
-        <parent link="camera_depth_frame" />
+        <origin xyz="0.017533 0.010995 0.012505" rpy="0 0 0" />
+        <parent link="camera_bottom_screw_frame" />
         <child link="camera_color_frame" />
         <axis xyz="0 0 0" />
@@ -238,6 +238,6 @@
     </link>
     <joint name="camera_color_optical_joint" type="fixed">
-        <origin xyz="0 0 0" rpy="-1.5707963267949 0 -1.5707963267949" />
-        <parent link="camera_color_frame" />
+        <origin xyz="0.017533 0.010995 0.012505" rpy="-1.5707963267949 0 -1.5707963267949" />
+        <parent link="camera_bottom_screw_frame" />
         <child link="camera_color_optical_frame" />
         <axis xyz="0 0 0" />
@@ -269,6 +269,6 @@
     </link>
     <joint name="camera_depth_joint" type="fixed">
-        <origin xyz="0 0 0" rpy="0 0 0" />
-        <parent link="camera_link" />
+        <origin xyz="0.01587 -0.025 0.0125" rpy="0 0 0" />
+        <parent link="camera_bottom_screw_frame" />
         <child link="camera_depth_frame" />
         <axis xyz="0 0 0" />
@@ -298,15 +298,15 @@
     </link>
     <joint name="camera_depth_optical_joint" type="fixed">
-        <origin xyz="0 0 0" rpy="-1.5707963267949 0 -1.5707963267949" />
-        <parent link="camera_depth_frame" />
+        <origin xyz="0.01587 -0.025 0.0125" rpy="-1.5707963267949 0 -1.5707963267949" />
+        <parent link="camera_bottom_screw_frame" />
         <child link="camera_depth_optical_frame" />
         <axis xyz="0 0 0" />
     </joint>
-    <!-- Alla fine aggiungi il joint che collega il Gemini alla testa -->
+    <!-- Joint che collega la Orbbec alla testa -->
     <joint name="head_camera_joint" type="fixed">
-      <!-- usa gli offset che avevi nel tuo URDF per la camera finta -->
-      <origin xyz="0.062346 -0.000241 0.034324" rpy="0 0 0"/>
-      <parent link="${parent_link}"/>
-      <child link="camera_bottom_screw_frame"/>
+        <!-- Offset della dummy camera - placeholder stilizzato in Fusion -->
+        <origin xyz="0.062346 -0.000241 0.034324" rpy="0 0 0"/>
+        <parent link="${parent_link}"/>
+        <child link="camera_link"/>
     </joint>
   </xacro:macro>

File: urdf/rakuda.xacro (robot description, xacro)
@@ -111,5 +111,7 @@
   </collision>
 </link>
+<!-- Chiama la macro che aggancia la Orbbec -->
 <xacro:gemini_335_336 parent_link="neck_pitch_link" />
+<!-- Link braccia -->
 <link name="l_link1">
   <inertial>

Commit message: removed collisions

File: urdf/gemini_335_336.urdf.xacro (robot description, xacro)
@@ -22,10 +22,4 @@
             </material>
         </visual>
-        <collision>
-            <origin xyz="0 0 0" rpy="0 0 0" />
-            <geometry>
-                <mesh filename="${mesh_path}camera_link.STL" />
-            </geometry>
-        </collision>
     </link>
     <link name="camera_bottom_screw_frame">
@@ -46,10 +40,4 @@
             </material>
         </visual>
-        <collision>
-            <origin xyz="0 0 0" rpy="0 0 0" />
-            <geometry>
-                <mesh filename="${mesh_path}camera_bottom_screw_frame.STL" />
-            </geometry>
-        </collision>
     </link>
     <joint name="camera_bottom_screw_frame_joint" type="fixed">
@@ -77,10 +65,4 @@
             </material>
         </visual>
-        <collision>
-            <origin xyz="0 0 0" rpy="0 0 0" />
-            <geometry>
-                <mesh filename="${mesh_path}camera_left_ir_frame.STL" />
-            </geometry>
-        </collision>
     </link>
     <joint name="camera_left_ir_joint" type="fixed">
@@ -107,10 +89,4 @@
             </material>
         </visual>
-        <collision>
-            <origin xyz="0 0 0" rpy="0 0 0" />
-            <geometry>
-                <mesh filename="${mesh_path}camera_left_ir_optical_frame.STL" />
-            </geometry>
-        </collision>
     </link>
     <joint name="camera_left_ir_optical_joint" type="fixed">
@@ -138,10 +114,4 @@
             </material>
         </visual>
-        <collision>
-            <origin xyz="0 0 0" rpy="0 0 0" />
-            <geometry>
-                <mesh filename="${mesh_path}camera_right_ir_frame.STL" />
-            </geometry>
-        </collision>
     </link>
     <joint name="camera_right_ir_joint" type="fixed">
@@ -168,10 +138,4 @@
             </material>
         </visual>
-        <collision>
-            <origin xyz="0 0 0" rpy="0 0 0" />
-            <geometry>
-                <mesh filename="${mesh_path}camera_right_ir_optical_frame.STL" />
-            </geometry>
-        </collision>
     </link>
     <joint name="camera_right_ir_optical_joint" type="fixed">
@@ -199,10 +163,4 @@
             </material>
         </visual>
-        <collision>
-            <origin xyz="0 0 0" rpy="0 0 0" />
-            <geometry>
-                <mesh filename="${mesh_path}camera_color_frame.STL" />
-            </geometry>
-        </collision>
     </link>
     <joint name="camera_color_joint" type="fixed">
@@ -230,10 +188,4 @@
             </material>
         </visual>
-        <collision>
-            <origin xyz="0 0 0" rpy="0 0 0" />
-            <geometry>
-                <mesh filename="${mesh_path}camera_color_optical_frame.STL" />
-            </geometry>
-        </collision>
     </link>
     <joint name="camera_color_optical_joint" type="fixed">
@@ -261,10 +213,4 @@
             </material>
         </visual>
-        <collision>
-            <origin xyz="0 0 0" rpy="0 0 0" />
-            <geometry>
-                <mesh filename="${mesh_path}camera_depth_frame.STL" />
-            </geometry>
-        </collision>
     </link>
     <joint name="camera_depth_joint" type="fixed">
@@ -290,10 +236,4 @@
             </material>
         </visual>
-        <collision>
-            <origin xyz="0 0 0" rpy="0 0 0" />
-            <geometry>
-                <mesh filename="${mesh_path}camera_depth_optical_frame.STL" />
-            </geometry>
-        </collision>
     </link>
     <joint name="camera_depth_optical_joint" type="fixed">

Commit message: removed camera_bottom_screw_frame

File: urdf/gemini_335_336.urdf.xacro (robot description, xacro)
@@ -23,28 +23,4 @@
         </visual>
     </link>
-    <link name="camera_bottom_screw_frame">
-        <inertial>
-            <origin xyz="0.00255168206289301 -0.00123934714960528 0.0118889875786098" rpy="0 0 0" />
-            <mass value="0.00564476880678651" />
-            <inertia ixx="3.07690693820862E-06" ixy="-1.85045956307764E-08"
-                ixz="-9.2792327175816E-09"
-                iyy="2.27632852811487E-07" iyz="1.65233162864392E-08" izz="2.93985735090777E-06" />
-        </inertial>
-        <visual>
-            <origin xyz="0 0 0" rpy="0 0 0" />
-            <geometry>
-                <mesh filename="${mesh_path}camera_bottom_screw_frame.STL" />
-            </geometry>
-            <material name="">
-                <color rgba="0.792156862745098 0.819607843137255 0.933333333333333 1" />
-            </material>
-        </visual>
-    </link>
-    <joint name="camera_bottom_screw_frame_joint" type="fixed">
-        <origin xyz="0 0 0" rpy="0 0 0" />
-        <parent link="camera_link" />
-        <child link="camera_bottom_screw_frame" />
-        <axis xyz="0 0 0" />
-    </joint>
     <link name="camera_left_ir_frame">
         <inertial>
@@ -68,5 +44,5 @@
     <joint name="camera_left_ir_joint" type="fixed">
         <origin xyz="0.01587 -0.025 0.0125" rpy="0 0 0" />
-        <parent link="camera_bottom_screw_frame" />
+        <parent link="camera_link" />
         <child link="camera_left_ir_frame" />
         <axis xyz="0 0 0" />
@@ -92,5 +68,5 @@
     <joint name="camera_left_ir_optical_joint" type="fixed">
         <origin xyz="0.01587 -0.025 0.0125" rpy="-1.5707963267949 0 -1.5707963267949" />
-        <parent link="camera_bottom_screw_frame" />
+        <parent link="camera_link" />
         <child link="camera_left_ir_optical_frame" />
         <axis xyz="0 0 0" />
@@ -117,5 +93,5 @@
     <joint name="camera_right_ir_joint" type="fixed">
         <origin xyz="0.01587 0.025 0.0125" rpy="0 0 0" />
-        <parent link="camera_bottom_screw_frame" />
+        <parent link="camera_link" />
         <child link="camera_right_ir_frame" />
         <axis xyz="0 0 0" />
@@ -141,5 +117,5 @@
     <joint name="camera_right_ir_optical_joint" type="fixed">
         <origin xyz="0.01587 0.025 0.0125" rpy="-1.5707963267949 0 -1.5707963267949" />
-        <parent link="camera_bottom_screw_frame" />
+        <parent link="camera_link" />
         <child link="camera_right_ir_optical_frame" />
         <axis xyz="0 0 0" />
@@ -166,5 +142,5 @@
     <joint name="camera_color_joint" type="fixed">
         <origin xyz="0.017533 0.010995 0.012505" rpy="0 0 0" />
-        <parent link="camera_bottom_screw_frame" />
+        <parent link="camera_link" />
         <child link="camera_color_frame" />
         <axis xyz="0 0 0" />
@@ -191,5 +167,5 @@
     <joint name="camera_color_optical_joint" type="fixed">
         <origin xyz="0.017533 0.010995 0.012505" rpy="-1.5707963267949 0 -1.5707963267949" />
-        <parent link="camera_bottom_screw_frame" />
+        <parent link="camera_link" />
         <child link="camera_color_optical_frame" />
         <axis xyz="0 0 0" />
@@ -216,5 +192,5 @@
     <joint name="camera_depth_joint" type="fixed">
         <origin xyz="0.01587 -0.025 0.0125" rpy="0 0 0" />
-        <parent link="camera_bottom_screw_frame" />
+        <parent link="camera_link" />
         <child link="camera_depth_frame" />
         <axis xyz="0 0 0" />
@@ -239,5 +215,5 @@
     <joint name="camera_depth_optical_joint" type="fixed">
         <origin xyz="0.01587 -0.025 0.0125" rpy="-1.5707963267949 0 -1.5707963267949" />
-        <parent link="camera_bottom_screw_frame" />
+        <parent link="camera_link" />
         <child link="camera_depth_optical_frame" />
         <axis xyz="0 0 0" />

Commit message: polished

File: urdf/gemini_335_336.urdf.xacro (robot description, xacro)
@@ -1,5 +1,5 @@
 <?xml version="1.0" encoding="utf-8"?>
 <robot xmlns:xacro="http://ros.org/wiki/xacro" name="gemini_335_336">
-  <!-- path per i mesh -->
+  <!-- path per i mesh della Orbbec -->
   <xacro:property name="mesh_path" value="package://orbbec_description/meshes/gemini335_336/" />
   <!-- macro che istanzia la Orbbec e la attacca al parent -->
@@ -220,5 +220,5 @@
     </joint>
     <!-- Joint che collega la Orbbec alla testa -->
-    <joint name="head_camera_joint" type="fixed">
+    <joint name="camera_joint" type="fixed">
         <!-- Offset della dummy camera - placeholder stilizzato in Fusion -->
         <origin xyz="0.062346 -0.000241 0.034324" rpy="0 0 0"/>

File: urdf/rakuda.xacro (robot description, xacro)
@@ -5,5 +5,5 @@
 <xacro:include filename="$(find rakuda_description)/urdf/rakuda.gazebo" />
 <xacro:include filename="$(find rakuda_description)/urdf/gemini_335_336.urdf.xacro" />
-<!-- Used for fixing robot 'base_link'  to Gazebo 'world' -->
+<!-- 'base_link'  to Gazebo 'world' -->
 <link name="world"/>
 <joint name="base_link_to_world_joint" type="fixed">
@@ -11,4 +11,5 @@
   <child link="base_link"/>
 </joint>
+<!-- Main links -->
 <link name="base_link">
   <inertial>
@@ -434,4 +435,5 @@
   </collision>
 </link>
+<!-- Joints -->
 <joint name="base_waist_joint" type="fixed">
   <origin xyz="0.0 0.0 0.302" rpy="0 0 0"/>

Commit message: refactoring

File: urdf/gemini_335_336.urdf.xacro (robot description, xacro)
@@ -222,5 +222,5 @@
     <joint name="camera_joint" type="fixed">
         <!-- Offset della dummy camera - placeholder stilizzato in Fusion -->
-        <origin xyz="0.062346 -0.000241 0.034324" rpy="0 0 0"/>
+        <origin xyz="0.057416 0.0 0.051447" rpy="0 0.099483767 0"/>
         <parent link="${parent_link}"/>
         <child link="camera_link"/>

File: urdf/rakuda.ros2_control.xacro (robot description, xacro)
@@ -142,6 +142,6 @@
         <!--<state_interface name="Present Current"/> -->
         <param name="Operating Mode">3</param>
-        <param name="Profile Velocity">40</param>
-        <param name="Profile Acceleration">20</param>
+        <param name="Profile Velocity">360</param>
+        <param name="Profile Acceleration">180</param>
         <param name="Position P Gain">800</param>
         <param name="Position I Gain">100</param>
@@ -158,6 +158,6 @@
         <!--<state_interface name="Present Current"/> -->
         <param name="Operating Mode">3</param>
-        <param name="Profile Velocity">40</param>
-        <param name="Profile Acceleration">20</param>
+        <param name="Profile Velocity">360</param>
+        <param name="Profile Acceleration">180</param>
         <param name="Position P Gain">800</param>
         <param name="Position I Gain">100</param>

File: urdf/rakuda.xacro (robot description, xacro)
@@ -94,19 +94,19 @@
 <link name="neck_pitch_link">
   <inertial>
-    <origin xyz="0.008434802102082811 -0.0003276428199875459 0.04341435318306919" rpy="0 0 0"/>
-    <mass value="0.2822100615108845"/>
-    <inertia ixx="695e-06" iyy="648e-06" izz="763e-06" ixy="0" iyz="-1e-06" ixz="42e-06"/>
+    <origin xyz="0.008396864265162956 -0.00019864066295206934 0.06883747797830841" rpy="0 0 0"/>
+    <mass value="0.42095197205408197"/>
+    <inertia ixx="4.708852" iyy="12.832797" izz="8.86896" ixy="0.006132" iyz="-0.007571" ixz="0.094646"/>
   </inertial>
   <visual>
     <origin xyz="0.0 -0.0001 -0.4606" rpy="0 0 0"/>
     <geometry>
-      <mesh filename="file://$(find rakuda_description)/meshes/visual/neck_pitch_link.stl" scale="0.001 0.001 0.001"/>
-    </geometry>
-    <material name="white"/>
-  </visual>
-  <collision>
-    <origin xyz="0.5 -0.0001 -0.4606" rpy="0 0 0"/>
-    <geometry>
-      <mesh filename="file://$(find rakuda_description)/meshes/collision/neck_pitch_link_collision.stl" scale="0.001 0.001 0.001"/>
+      <mesh filename="file://$(find rakuda_description)/meshes/visual/neck_pitch_link_ap.stl" scale="0.001 0.001 0.001"/>
+    </geometry>
+    <material name="white"/>
+  </visual>
+  <collision>
+    <origin xyz="0.0 -0.0001 -0.4606" rpy="0 0 0"/>
+    <geometry>
+      <mesh filename="file://$(find rakuda_description)/meshes/collision/neck_pitch_link_ap_collision.stl" scale="0.001 0.001 0.001"/>
     </geometry>
   </collision>
@@ -114,5 +114,5 @@
 <!-- Chiama la macro che aggancia la Orbbec -->
 <xacro:gemini_335_336 parent_link="neck_pitch_link" />
-<!-- Chiama la macro che aggancia il ros control: Inserire il numero di Dynamixel -->
+<!-- Chiama la macro che aggancia il ros control: Inserire il numero totale di Dynamixel -->
 <xacro:property name="dof" value="17"/>
 <xacro:include filename="rakuda.ros2_control.xacro"/>
@@ -449,5 +449,5 @@
   <parent link="waist_link"/>
   <child link="torso_link"/>
-  <axis xyz="0.0 0.0 -1.0"/>
+  <axis xyz="0.0 0.0 1.0"/>
   <limit upper="1.396263" lower="-1.396263" effort="100" velocity="100"/>
   <dynamics damping="1.0e-6" friction="0.8"/>
@@ -458,5 +458,6 @@
   <child link="neck_yaw_link"/>
   <axis xyz="0.0 0.0 1.0"/>
-  <limit upper="1.22173" lower="-1.22173" effort="100" velocity="100"/>
+  <!-- Sciurus17 limit upper="1.22173" lower="-1.22173" effort="100" velocity="100"/ -->
+  <limit upper="0.660" lower="-0.660" effort="100" velocity="100"/>
   <dynamics damping="1.0e-6" friction="0.8"/>
 </joint>
@@ -466,5 +467,6 @@
   <child link="neck_pitch_link"/>
   <axis xyz="0.0 -1.0 0.0"/>
-  <limit upper="0.610865" lower="-0.872665" effort="100" velocity="100"/>
+  <!-- Sciurus17 limit upper="0.610865" lower="-0.872665" effort="100" velocity="100" -->
+  <limit upper="0.5235" lower="-0.530" effort="100" velocity="100"/>
   <dynamics damping="1.0e-6" friction="0.8"/>
 </joint>

Commit message: variabilizzazione testa

File: urdf/gemini_335_336.urdf.xacro (robot description, xacro)
@@ -4,5 +4,5 @@
   <xacro:property name="mesh_path" value="package://orbbec_description/meshes/gemini335_336/" />
   <!-- macro che istanzia la Orbbec e la attacca al parent -->
-  <xacro:macro name="gemini_335_336" params="parent_link">
+  <xacro:macro name="gemini_335_336" params="parent_link xyz_joint_origin rpy_joint_origin">
     <link name="camera_link">
         <inertial>
@@ -222,5 +222,5 @@
     <joint name="camera_joint" type="fixed">
         <!-- Offset della dummy camera - placeholder stilizzato in Fusion -->
-        <origin xyz="0.057416 0.0 0.051447" rpy="0 0.099483767 0"/>
+        <origin xyz="${xyz_joint_origin}" rpy="${rpy_joint_origin}"/>
         <parent link="${parent_link}"/>
         <child link="camera_link"/>

File: urdf/rakuda.xacro (robot description, xacro)
@@ -1,8 +1,20 @@
 <?xml version="1.0" ?>
 <robot name="rakuda" xmlns:xacro="http://www.ros.org/wiki/xacro">
+<!-- Variabile testa -->
+<xacro:arg name="head_type" default="apollo"/>
+<xacro:property name="head_type" value="$(arg head_type)"/>
 <xacro:include filename="$(find rakuda_description)/urdf/materials.xacro" />
 <xacro:include filename="$(find rakuda_description)/urdf/rakuda.ros2_control.xacro" />
 <xacro:include filename="$(find rakuda_description)/urdf/rakuda.gazebo" />
-<xacro:include filename="$(find rakuda_description)/urdf/gemini_335_336.urdf.xacro" />
+<!-- Teste disponibili -->
+<xacro:include filename="$(find rakuda_description)/urdf/head_apollo.urdf.xacro"/>
+<xacro:include filename="$(find rakuda_description)/urdf/head_sciurus.urdf.xacro"/>
+<!-- Scelta della testa da caricare -->
+<xacro:if value="${head_type == 'apollo'}">
+  <xacro:head_apollo parent_link="neck_yaw_link"/>
+</xacro:if>
+<xacro:if value="${head_type == 'sciurus'}">
+  <xacro:head_sciurus parent_link="neck_yaw_link"/>
+</xacro:if>
 <!-- 'base_link'  to Gazebo 'world' -->
 <link name="world"/>
@@ -92,26 +104,4 @@
   </collision>
 </link>
-<link name="neck_pitch_link">
-  <inertial>
-    <origin xyz="0.008396864265162956 -0.00019864066295206934 0.06883747797830841" rpy="0 0 0"/>
-    <mass value="0.42095197205408197"/>
-    <inertia ixx="4.708852" iyy="12.832797" izz="8.86896" ixy="0.006132" iyz="-0.007571" ixz="0.094646"/>
-  </inertial>
-  <visual>
-    <origin xyz="0.0 -0.0001 -0.4606" rpy="0 0 0"/>
-    <geometry>
-      <mesh filename="file://$(find rakuda_description)/meshes/visual/neck_pitch_link_ap.stl" scale="0.001 0.001 0.001"/>
-    </geometry>
-    <material name="white"/>
-  </visual>
-  <collision>
-    <origin xyz="0.0 -0.0001 -0.4606" rpy="0 0 0"/>
-    <geometry>
-      <mesh filename="file://$(find rakuda_description)/meshes/collision/neck_pitch_link_ap_collision.stl" scale="0.001 0.001 0.001"/>
-    </geometry>
-  </collision>
-</link>
-<!-- Chiama la macro che aggancia la Orbbec -->
-<xacro:gemini_335_336 parent_link="neck_pitch_link" />
 <!-- Chiama la macro che aggancia il ros control: Inserire il numero totale di Dynamixel -->
 <xacro:property name="dof" value="17"/>
@@ -462,13 +452,4 @@
   <dynamics damping="1.0e-6" friction="0.8"/>
 </joint>
-<joint name="neck_pitch_joint" type="revolute">
-  <origin xyz="-0.0 0.0001 0.02655" rpy="0 0 0"/>
-  <parent link="neck_yaw_link"/>
-  <child link="neck_pitch_link"/>
-  <axis xyz="0.0 -1.0 0.0"/>
-  <!-- Sciurus17 limit upper="0.610865" lower="-0.872665" effort="100" velocity="100" -->
-  <limit upper="0.5235" lower="-0.530" effort="100" velocity="100"/>
-  <dynamics damping="1.0e-6" friction="0.8"/>
-</joint>
 <joint name="l_arm_joint1" type="revolute">
   <origin xyz="0.0 0.0826 0.0861" rpy="0 0 0"/>

Commit message: Update visual origin position in URDF file
Era:    
<link name="camera_left_ir_frame">
        <visual>
            <origin xyz="-25 0 0" rpy="0 0 0" />

File: urdf/gemini_335_336.urdf.xacro (robot description, xacro)
@@ -33,5 +33,5 @@
         </inertial>
         <visual>
-            <origin xyz="-25 0 0" rpy="0 0 0" />
+            <origin xyz="0 0 0" rpy="0 0 0" />
             <geometry>
                 <mesh filename="${mesh_path}camera_left_ir_frame.STL" />
