Commit message: Remove unused axis definitions from fixed joints

File: urdf/gemini_335_336.urdf.xacro (robot description, xacro)
@@ -46,5 +46,4 @@
         <parent link="camera_link" />
         <child link="camera_left_ir_frame" />
-        <axis xyz="0 0 0" />
     </joint>
     <link name="camera_left_ir_optical_frame">
@@ -70,5 +69,4 @@
         <parent link="camera_link" />
         <child link="camera_left_ir_optical_frame" />
-        <axis xyz="0 0 0" />
     </joint>
     <link name="camera_right_ir_frame">
@@ -95,5 +93,4 @@
         <parent link="camera_link" />
         <child link="camera_right_ir_frame" />
-        <axis xyz="0 0 0" />
     </joint>
     <link name="camera_right_ir_optical_frame">
@@ -119,5 +116,4 @@
         <parent link="camera_link" />
         <child link="camera_right_ir_optical_frame" />
-        <axis xyz="0 0 0" />
     </joint>
     <link name="camera_color_frame">
@@ -144,5 +140,4 @@
         <parent link="camera_link" />
         <child link="camera_color_frame" />
-        <axis xyz="0 0 0" />
     </joint>
     <link name="camera_color_optical_frame">
@@ -169,5 +164,4 @@
         <parent link="camera_link" />
         <child link="camera_color_optical_frame" />
-        <axis xyz="0 0 0" />
     </joint>
     <link name="camera_depth_frame">
@@ -194,5 +188,4 @@
         <parent link="camera_link" />
         <child link="camera_depth_frame" />
-        <axis xyz="0 0 0" />
     </joint>
     <link name="camera_depth_optical_frame">
@@ -217,5 +210,4 @@
         <parent link="camera_link" />
         <child link="camera_depth_optical_frame" />
-        <axis xyz="0 0 0" />
     </joint>
     <!-- Joint che collega la Orbbec alla testa -->

Commit message: preparation fopr moveit

File: urdf/gemini_335_336.urdf.xacro (robot description, xacro)
@@ -22,4 +22,7 @@
             </material>
         </visual>
+        <collision>
+            <origin xyz="0 0 0" rpy="0 0 0" />
+        </collision>
     </link>
     <link name="camera_left_ir_frame">
@@ -41,4 +44,7 @@
             </material>
         </visual>
+        <collision>
+            <origin xyz="0 0 0" rpy="0 0 0" />
+        </collision>
     </link>
     <joint name="camera_left_ir_joint" type="fixed">
@@ -64,4 +70,7 @@
             </material>
         </visual>
+        <collision>
+            <origin xyz="0 0 0" rpy="0 0 0" />
+        </collision>
     </link>
     <joint name="camera_left_ir_optical_joint" type="fixed">
@@ -88,4 +97,7 @@
             </material>
         </visual>
+        <collision>
+            <origin xyz="0 0 0" rpy="0 0 0" />
+        </collision>
     </link>
     <joint name="camera_right_ir_joint" type="fixed">
@@ -111,4 +123,7 @@
             </material>
         </visual>
+        <collision>
+            <origin xyz="0 0 0" rpy="0 0 0" />
+        </collision>
     </link>
     <joint name="camera_right_ir_optical_joint" type="fixed">
@@ -135,4 +150,7 @@
             </material>
         </visual>
+        <collision>
+            <origin xyz="0 0 0" rpy="0 0 0" />
+        </collision>
     </link>
     <joint name="camera_color_joint" type="fixed">
@@ -159,4 +177,7 @@
             </material>
         </visual>
+        <collision>
+            <origin xyz="0 0 0" rpy="0 0 0" />
+        </collision>
     </link>
     <joint name="camera_color_optical_joint" type="fixed">
@@ -183,4 +204,7 @@
             </material>
         </visual>
+        <collision>
+            <origin xyz="0 0 0" rpy="0 0 0" />
+        </collision>
     </link>
     <joint name="camera_depth_joint" type="fixed">
@@ -205,4 +229,7 @@
             </material>
         </visual>
+        <collision>
+            <origin xyz="0 0 0" rpy="0 0 0" />
+        </collision>
     </link>
     <joint name="camera_depth_optical_joint" type="fixed">

File: urdf/rakuda.ros2_control.xacro (robot description, xacro)
@@ -9,7 +9,13 @@
     ])}
   </xacro:macro>
-  <xacro:macro name="rakuda_ros2_control_settings" params="dof">
-    <ros2_control name="DynamixelTorsoHeadSystem" type="system">
-      <hardware>
+<xacro:macro name="rakuda_ros2_control_settings" params="dof use_mock_hardware:=true mock_sensor_commands:=true">
+  <!-- (consiglio) rinomina per non confondere i log -->
+  <ros2_control name="RakudaSystem" type="system">
+    <hardware>
+      <xacro:if value="${use_mock_hardware}">
+        <plugin>mock_components/GenericSystem</plugin>
+        <param name="mock_sensor_commands">${mock_sensor_commands}</param>
+      </xacro:if>
+      <xacro:unless value="${use_mock_hardware}">
         <plugin>dynamixel_hardware_interface/DynamixelHardware</plugin>
         <param name="port_name">/dev/ttyU2D2</param>
@@ -27,4 +33,5 @@
         <param name="reboot_dxl_srv_name">dynamixel_hardware_interface/reboot_dxl</param>
         <param name="set_dxl_torque_srv_name">dynamixel_hardware_interface/set_dxl_torque</param>
+        </xacro:unless>
       </hardware>
       <joint name="waist_yaw_joint">

File: urdf/rakuda.urdf (robot description, URDF)
Before this commit: robot rakuda, 31 links, 30 joints
Joints:
- joint l_arm_joint1: limit lower=-2.96706 upper=0.0 effort=100 velocity=100 -> lower=-2.96706 upper=0.0 effort=100.0 velocity=4.8
- joint l_arm_joint2: limit lower=-0.0 upper=1.570796 effort=100 velocity=100 -> lower=-0.0 upper=1.570796 effort=100.0 velocity=4.8
- joint l_arm_joint3: limit lower=-1.396263 upper=1.396263 effort=100 velocity=100 -> lower=-1.396263 upper=1.396263 effort=100.0 velocity=4.8
- joint l_arm_joint4: limit lower=-2.356194 upper=0.174533 effort=100 velocity=100 -> lower=-2.356194 upper=0.174533 effort=100.0 velocity=4.8
- joint l_arm_joint5: limit lower=-1.570796 upper=1.570796 effort=100 velocity=100 -> lower=-1.570796 upper=1.570796 effort=100.0 velocity=4.8
- joint l_arm_joint6: limit lower=-1.396263 upper=1.396263 effort=100 velocity=100 -> lower=-1.396263 upper=1.396263 effort=100.0 velocity=4.8
- joint l_gripper_joint: limit lower=0.0 upper=1.22173 effort=100 velocity=100 -> lower=0.0 upper=1.22173 effort=100.0 velocity=4.8
- joint neck_yaw_joint: limit lower=-0.660 upper=0.660 effort=100 velocity=100 -> lower=-0.660 upper=0.660 effort=100.0 velocity=4.8
- joint r_arm_joint1: limit lower=0.0 upper=2.96706 effort=100 velocity=100 -> lower=0.0 upper=2.96706 effort=100.0 velocity=4.8
- joint r_arm_joint2: limit lower=-1.570796 upper=0.0 effort=100 velocity=100 -> lower=-1.570796 upper=0.0 effort=100.0 velocity=4.8
- joint r_arm_joint3: limit lower=-1.396263 upper=1.396263 effort=100 velocity=100 -> lower=-1.396263 upper=1.396263 effort=100.0 velocity=4.8
- joint r_arm_joint4: limit lower=-0.174533 upper=2.356194 effort=100 velocity=100 -> lower=-0.174533 upper=2.356194 effort=100.0 velocity=4.8
- joint r_arm_joint5: limit lower=-1.570796 upper=1.570796 effort=100 velocity=100 -> lower=-1.570796 upper=1.570796 effort=100.0 velocity=4.8
- joint r_arm_joint6: limit lower=-1.396263 upper=1.396263 effort=100 velocity=100 -> lower=-1.396263 upper=1.396263 effort=100.0 velocity=4.8
- joint r_gripper_joint: limit lower=-1.22173 upper=0.0 effort=100 velocity=100 -> lower=-1.22173 upper=0.0 effort=100.0 velocity=4.8
- joint waist_yaw_joint: limit lower=-1.396263 upper=1.396263 effort=100 velocity=100 -> lower=-1.396263 upper=1.396263 effort=100.0 velocity=4.8

File: urdf/rakuda.urdf.xacro (robot description, xacro)
@@ -3,9 +3,10 @@
 <!-- Variabile testa anche inseribile in file launch-->
 <xacro:arg name="head_type" default="apollo"/>
+<xacro:arg name="use_mock_hardware" default="false"/>
+<xacro:arg name="mock_sensor_commands" default="false"/>
 <xacro:property name="head_type" value="$(arg head_type)"/>
 <xacro:include filename="$(find rakuda_description)/urdf/gemini_335_336.urdf.xacro" />
 <xacro:include filename="$(find rakuda_description)/urdf/materials.xacro" />
 <xacro:include filename="$(find rakuda_description)/urdf/rakuda.ros2_control.xacro" />
-<xacro:include filename="$(find rakuda_description)/urdf/rakuda.gazebo" />
 <!-- Teste disponibili -->
 <xacro:include filename="$(find rakuda_description)/urdf/head_apollo.urdf.xacro"/>
@@ -115,5 +116,8 @@
 <!-- Chiama la macro che aggancia il ros control: Inserire il numero totale di Dynamixel -->
 <xacro:property name="dof" value="17"/>
-<xacro:rakuda_ros2_control_settings dof="${dof}"/>
+<xacro:rakuda_ros2_control_settings
+  dof="${dof}"
+  use_mock_hardware="$(arg use_mock_hardware)"
+  mock_sensor_commands="$(arg mock_sensor_commands)"/>
 <!-- Link braccia -->
 <link name="l_link1">

Commit message: update

File: urdf/gemini_335_336.urdf.xacro (robot description, xacro)
@@ -24,4 +24,7 @@
         <collision>
             <origin xyz="0 0 0" rpy="0 0 0" />
+            <geometry>
+                <mesh filename="${mesh_path}camera_link.STL" />
+            </geometry>
         </collision>
     </link>
@@ -46,4 +49,7 @@
         <collision>
             <origin xyz="0 0 0" rpy="0 0 0" />
+            <geometry>
+                <mesh filename="${mesh_path}camera_left_ir_frame.STL" />
+            </geometry>
         </collision>
     </link>
@@ -72,4 +78,7 @@
         <collision>
             <origin xyz="0 0 0" rpy="0 0 0" />
+            <geometry>
+                <mesh filename="${mesh_path}camera_left_ir_optical_frame.STL" />
+            </geometry>
         </collision>
     </link>
@@ -99,4 +108,7 @@
         <collision>
             <origin xyz="0 0 0" rpy="0 0 0" />
+            <geometry>
+                <mesh filename="${mesh_path}camera_right_ir_frame.STL" />
+            </geometry>
         </collision>
     </link>
@@ -125,4 +137,7 @@
         <collision>
             <origin xyz="0 0 0" rpy="0 0 0" />
+            <geometry>
+                <mesh filename="${mesh_path}camera_right_ir_optical_frame.STL" />
+            </geometry>
         </collision>
     </link>
@@ -152,4 +167,7 @@
         <collision>
             <origin xyz="0 0 0" rpy="0 0 0" />
+            <geometry>
+                <mesh filename="${mesh_path}camera_color_frame.STL" />
+            </geometry>
         </collision>
     </link>
@@ -179,4 +197,7 @@
         <collision>
             <origin xyz="0 0 0" rpy="0 0 0" />
+            <geometry>
+                <mesh filename="${mesh_path}camera_color_optical_frame.STL" />
+            </geometry>
         </collision>
     </link>
@@ -206,4 +227,7 @@
         <collision>
             <origin xyz="0 0 0" rpy="0 0 0" />
+            <geometry>
+                <mesh filename="${mesh_path}camera_depth_frame.STL" />
+            </geometry>
         </collision>
     </link>
@@ -231,4 +255,7 @@
         <collision>
             <origin xyz="0 0 0" rpy="0 0 0" />
+            <geometry>
+                <mesh filename="${mesh_path}camera_depth_optical_frame.STL" />
+            </geometry>
         </collision>
     </link>

File: urdf/rakuda.urdf (robot description, URDF)
Before this commit: robot rakuda, 31 links, 30 joints
Links:
- link camera_color_frame: geometry collision mesh filename=package://orbbec_description/meshes/gemini335_336/camera_co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; visual mesh filename=package://orbbec_description/meshes/gemini335_336/camera_co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
- link camera_color_optical_frame: geometry collision mesh filename=package://orbbec_description/meshes/gemini335_336/camera_co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; visual mesh filename=package://orbbec_description/meshes/gemini335_336/camera_co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
- link camera_depth_frame: geometry collision mesh filename=package://orbbec_description/meshes/gemini335_336/camera_de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; visual mesh filename=package://orbbec_description/meshes/gemini335_336/camera_de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
- link camera_depth_optical_frame: geometry collision mesh filename=package://orbbec_description/meshes/gemini335_336/camera_de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; visual mesh filename=package://orbbec_description/meshes/gemini335_336/camera_de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
- link camera_left_ir_frame: geometry collision mesh filename=package://orbbec_description/meshes/gemini335_336/camera_le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; visual mesh filename=package://orbbec_description/meshes/gemini335_336/camera_le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
- link camera_left_ir_optical_frame: geometry collision mesh filename=package://orbbec_description/meshes/gemini335_336/camera_le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; visual mesh filename=package://orbbec_description/meshes/gemini335_336/camera_le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
- link camera_link: geometry collision mesh filename=package://orbbec_description/meshes/gemini335_336/camera_li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; visual mesh filename=package://orbbec_description/meshes/gemini335_336/camera_li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
- link camera_right_ir_frame: geometry collision mesh filename=package://orbbec_description/meshes/gemini335_336/camera_ri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; visual mesh filename=package://orbbec_description/meshes/gemini335_336/camera_ri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
- link camera_right_ir_optical_frame: geometry collision mesh filename=package://orbbec_description/meshes/gemini335_336/camera_ri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; visual mesh filename=package://orbbec_description/meshes/gemini335_336/camera_ri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
