Commit message: refactoring

File: urdf/head_apollo.urdf.xacro (robot description, xacro)
@@ -5,31 +5,30 @@
     <xacro:macro name="head_apollo" params="parent_link">
     <link name="neck_pitch_link">
-    <inertial>
-    <origin xyz="0.008396864265162956 -0.00019864066295206934 0.06883747797830841" rpy="0 0 0"/>
-    <mass value="0.42095197205408197"/>
-    <inertia ixx="4.708852" iyy="12.832797" izz="8.86896" ixy="0.006132" iyz="-0.007571" ixz="0.094646"/>
-    </inertial>
-    <visual>
-    <origin xyz="0.0 -0.0001 -0.4606" rpy="0 0 0"/>
-    <geometry>
-      <mesh filename="file://$(find rakuda_description)/meshes/visual/neck_pitch_link_ap.stl" scale="0.001 0.001 0.001"/>
-    </geometry>
-    <material name="white"/>
-    </visual>
-    <collision>
-    <origin xyz="0.0 -0.0001 -0.4606" rpy="0 0 0"/>
-    <geometry>
-      <mesh filename="file://$(find rakuda_description)/meshes/collision/neck_pitch_link_ap_collision.stl" scale="0.001 0.001 0.001"/>
-    </geometry>
-    </collision>
+      <inertial>
+        <origin xyz="0.008396864265162956 -0.00019864066295206934 0.06883747797830841" rpy="0 0 0"/>
+        <mass value="0.42095197205408197"/>
+        <inertia ixx="4.708852" iyy="12.832797" izz="8.86896" ixy="0.006132" iyz="-0.007571" ixz="0.094646"/>
+      </inertial>
+      <visual>
+        <origin xyz="0.0 -0.0001 -0.4606" rpy="0 0 0"/>
+        <geometry>
+          <mesh filename="file://$(find rakuda_description)/meshes/visual/neck_pitch_link_ap.stl" scale="0.001 0.001 0.001"/>
+        </geometry>
+        <material name="white"/>
+      </visual>
+      <collision>
+        <origin xyz="0.0 -0.0001 -0.4606" rpy="0 0 0"/>
+        <geometry>
+          <mesh filename="file://$(find rakuda_description)/meshes/collision/neck_pitch_link_ap_collision.stl" scale="0.001 0.001 0.001"/>
+        </geometry>
+      </collision>
     </link>
     <joint name="neck_pitch_joint" type="revolute">
-        <origin xyz="-0.0 0.0001 0.02655" rpy="0 0 0"/>
-        <parent link="${parent_link}"/>
-        <child link="neck_pitch_link"/>
-        <axis xyz="0.0 -1.0 0.0"/>
-        <!-- Sciurus17 limit upper="0.610865" lower="-0.872665" effort="100" velocity="100" -->
-        <limit upper="0.5235" lower="-0.530" effort="100" velocity="100"/>
-        <dynamics damping="1.0e-6" friction="0.8"/>
+      <origin xyz="-0.0 0.0001 0.02655" rpy="0 0 0"/>
+      <parent link="${parent_link}"/>
+      <child link="neck_pitch_link"/>
+      <axis xyz="0.0 -1.0 0.0"/>
+      <limit upper="0.5235" lower="-0.530" effort="100" velocity="100"/>
+      <dynamics damping="1.0e-6" friction="0.8"/>
     </joint>
     <!-- Chiama la macro che aggancia la Orbbec -->

Commit message: cleansing

File: urdf/head_apollo.urdf.xacro (robot description, xacro)
@@ -5,7 +5,7 @@
     <link name="neck_pitch_link">
       <inertial>
-        <origin xyz="0.008396864265162956 -0.00019864066295206934 0.06883747797830841" rpy="0 0 0"/>
-        <mass value="0.42095197205408197"/>
-        <inertia ixx="4.708852" iyy="12.832797" izz="8.86896" ixy="0.006132" iyz="-0.007571" ixz="0.094646"/>
+        <origin xyz="0.00803 -0.000092 0.530156" rpy="0 0 0"/>
+        <mass value="0.396256"/>
+        <inertia ixx="8130e-06" ixy="1.134e-06" ixz="720.5e-06" iyy="12790e-06" iyz="-0.602e-06" izz="11010e-06"/>
       </inertial>
       <visual>
@@ -28,5 +28,5 @@
       <child link="neck_pitch_link"/>
       <axis xyz="0.0 -1.0 0.0"/>
-      <limit upper="0.5235" lower="-0.530" effort="100" velocity="100"/>
+      <limit upper="0.5235" lower="-0.530" effort="4.1" velocity="4.8"/>
       <dynamics damping="1.0e-6" friction="0.8"/>
     </joint>

File: urdf/rakuda.urdf.xacro (robot description, xacro)
@@ -452,5 +452,5 @@
   <child link="torso_link"/>
   <axis xyz="0.0 0.0 1.0"/>
-  <limit upper="1.396263" lower="-1.396263" effort="100.0" velocity="4.8"/>
+  <limit upper="1.396263" lower="-1.396263" effort="10.0" velocity="4.8"/>
   <dynamics damping="1.0e-6" friction="0.8"/>
 </joint>
@@ -461,5 +461,5 @@
   <axis xyz="0.0 0.0 1.0"/>
   <!-- Sciurus17 limit upper="1.22173" lower="-1.22173" effort="100.0" velocity="4.8"/ -->
-  <limit upper="0.660" lower="-0.660" effort="100.0" velocity="4.8"/>
+  <limit upper="0.660" lower="-0.660" effort="4.1" velocity="4.8"/>
   <dynamics damping="1.0e-6" friction="0.8"/>
 </joint>
@@ -469,5 +469,5 @@
   <child link="l_link1"/>
   <axis xyz="0.0 1.0 0.0"/>
-  <limit upper="0.0" lower="-2.96706" effort="100.0" velocity="4.8"/>
+  <limit upper="0.0" lower="-2.96706" effort="10.0" velocity="4.8"/>
   <dynamics damping="1.0e-6" friction="0.8"/>
 </joint>
@@ -477,5 +477,5 @@
   <child link="r_link1"/>
   <axis xyz="0.0 -1.0 0.0"/>
-  <limit upper="2.96706" lower="0.0" effort="100.0" velocity="4.8"/>
+  <limit upper="2.96706" lower="0.0" effort="10.0" velocity="4.8"/>
   <dynamics damping="1.0e-6" friction="0.8"/>
 </joint>
@@ -485,5 +485,5 @@
   <child link="l_link2"/>
   <axis xyz="1.0 0.0 0.0"/>
-  <limit upper="1.570796" lower="-0.0" effort="100.0" velocity="4.8"/>
+  <limit upper="1.570796" lower="-0.0" effort="10.0" velocity="4.8"/>
   <dynamics damping="1.0e-6" friction="0.8"/>
 </joint>
@@ -493,5 +493,5 @@
   <child link="r_link2"/>
   <axis xyz="1.0 0.0 0.0"/>
-  <limit upper="0.0" lower="-1.570796" effort="100.0" velocity="4.8"/>
+  <limit upper="0.0" lower="-1.570796" effort="10.0" velocity="4.8"/>
   <dynamics damping="1.0e-6" friction="0.8"/>
 </joint>
@@ -501,5 +501,5 @@
   <child link="l_link3"/>
   <axis xyz="0.0 0.0 -1.0"/>
-  <limit upper="1.396263" lower="-1.396263" effort="100.0" velocity="4.8"/>
+  <limit upper="1.396263" lower="-1.396263" effort="4.1" velocity="4.8"/>
   <dynamics damping="1.0e-6" friction="0.8"/>
 </joint>
@@ -509,5 +509,5 @@
   <child link="r_link3"/>
   <axis xyz="0.0 0.0 -1.0"/>
-  <limit upper="1.396263" lower="-1.396263" effort="100.0" velocity="4.8"/>
+  <limit upper="1.396263" lower="-1.396263" effort="4.1" velocity="4.8"/>
   <dynamics damping="1.0e-6" friction="0.8"/>
 </joint>
@@ -517,5 +517,5 @@
   <child link="l_link4"/>
   <axis xyz="0.0 1.0 0.0"/>
-  <limit upper="0.174533" lower="-2.356194" effort="100.0" velocity="4.8"/>
+  <limit upper="0.174533" lower="-2.356194" effort="4.1" velocity="4.8"/>
   <dynamics damping="1.0e-6" friction="0.8"/>
 </joint>
@@ -525,5 +525,5 @@
   <child link="r_link4"/>
   <axis xyz="0.0 -1.0 0.0"/>
-  <limit upper="2.356194" lower="-0.174533" effort="100.0" velocity="4.8"/>
+  <limit upper="2.356194" lower="-0.174533" effort="4.1" velocity="4.8"/>
   <dynamics damping="1.0e-6" friction="0.8"/>
 </joint>
@@ -533,5 +533,5 @@
   <child link="l_link5"/>
   <axis xyz="0.0 0.0 -1.0"/>
-  <limit upper="1.570796" lower="-1.570796" effort="100.0" velocity="4.8"/>
+  <limit upper="1.570796" lower="-1.570796" effort="4.1" velocity="4.8"/>
   <dynamics damping="1.0e-6" friction="0.8"/>
 </joint>
@@ -541,5 +541,5 @@
   <child link="r_link5"/>
   <axis xyz="0.0 0.0 -1.0"/>
-  <limit upper="1.570796" lower="-1.570796" effort="100.0" velocity="4.8"/>
+  <limit upper="1.570796" lower="-1.570796" effort="4.1" velocity="4.8"/>
   <dynamics damping="1.0e-6" friction="0.8"/>
 </joint>
@@ -549,5 +549,5 @@
   <child link="r_link6"/>
   <axis xyz="0.0 -1.0 0.0"/>
-  <limit upper="1.396263" lower="-1.396263" effort="100.0" velocity="4.8"/>
+  <limit upper="1.396263" lower="-1.396263" effort="4.1" velocity="4.8"/>
   <dynamics damping="1.0e-6" friction="0.8"/>
 </joint>
@@ -557,5 +557,5 @@
   <child link="l_link6"/>
   <axis xyz="0.0 1.0 0.0"/>
-  <limit upper="1.396263" lower="-1.396263" effort="100.0" velocity="4.8"/>
+  <limit upper="1.396263" lower="-1.396263" effort="4.1" velocity="4.8"/>
   <dynamics damping="1.0e-6" friction="0.8"/>
 </joint>
@@ -565,10 +565,10 @@
   <child link="r_gripper_a"/>
   <axis xyz="1.0 0.0 0.0"/>
-  <limit upper="0.0" lower="-1.22173" effort="100.0" velocity="4.8"/>
+  <limit upper="0.0" lower="-1.22173" effort="1.5" velocity="4.8"/>
   <dynamics damping="1.0e-6" friction="0.8"/>
 </joint>
 <joint name="r_gripper_mimic_joint" type="revolute">
   <origin xyz="0.0 0.008 -0.0423" rpy="0 0 0"/>
-  <limit lower="-1.0" upper="0.01" effort="10" velocity="1.0"/>
+  <limit lower="-1.0" upper="0.01" effort="1.5" velocity="1.0"/>
   <parent link="r_link6"/>
   <child link="r_gripper_b"/>
@@ -581,10 +581,10 @@
   <child link="l_gripper_a"/>
   <axis xyz="1.0 0.0 0.0"/>
-  <limit upper="1.22173" lower="0.0" effort="100.0" velocity="4.8"/>
+  <limit upper="1.22173" lower="0.0" effort="1.5" velocity="4.8"/>
   <dynamics damping="1.0e-6" friction="0.8"/>
 </joint>
 <joint name="l_gripper_mimic_joint" type="revolute">
   <origin xyz="0.0 -0.008 -0.0423" rpy="0 0 0"/>
-  <limit lower="-0.01" upper="1.0" effort="10" velocity="1.0"/>
+  <limit lower="-0.01" upper="1.0" effort="1.5" velocity="1.0"/>
   <parent link="l_link6"/>
   <child link="l_gripper_b"/>
