Commit message: upload waist test

File: urdf/rakuda.ros2_control.xacro (robot description, xacro)
@@ -1,3 +1,205 @@
-<?xml version="1.0" ?>
-<robot name="rakuda" xmlns:xacro="http://www.ros.org/wiki/xacro" >
+<?xml version="1.0"?>
+<robot xmlns:xacro="http://www.ros.org/wiki/xacro">
+  <xacro:macro name="rakuda_ros2_control_settings">
+    <!-- TODO: inserire il parametro nel main cxaxroJoint che collega la Orbbec alla testa -->
+    <ros2_control name="rakuda" type="system">
+      <hardware>
+          <plugin>sciurus17_hardware/Sciurus17Hardware</plugin>
+          <param name="port_name">${PORT_NAME}</param>
+          <param name="baudrate">${BAUDRATE}</param>
+          <param name="timeout_seconds">${TIMEOUT_SECONDS}</param>
+          <param name="manipulator_config_file_path">${MANIPULATOR_CONFIG_FILE_PATH}</param>
+      </hardware>
+      <joint name="${NAME_JOINT_BODY}">
+        <command_interface name="position">
+          <param name="min">${JOINT_BODY_LOWER_LIMIT}</param>
+          <param name="max">${JOINT_BODY_UPPER_LIMIT}</param>
+        </command_interface>
+        <state_interface name="position"/>
+        <state_interface name="velocity"/>
+        <state_interface name="effort"/>
+        <param name="current_to_effort">3.60</param>
+      </joint>
+      <joint name="${NAME_JOINT_NECK_1}">
+        <command_interface name="position">
+          <param name="min">${JOINT_NECK_1_LOWER_LIMIT}</param>
+          <param name="max">${JOINT_NECK_1_UPPER_LIMIT}</param>
+        </command_interface>
+        <state_interface name="position"/>
+        <state_interface name="velocity"/>
+        <state_interface name="effort"/>
+        <param name="current_to_effort">2.20</param>
+      </joint>
+      <joint name="${NAME_JOINT_NECK_2}">
+        <command_interface name="position">
+          <param name="min">${JOINT_NECK_2_LOWER_LIMIT}</param>
+          <param name="max">${JOINT_NECK_2_UPPER_LIMIT}</param>
+        </command_interface>
+        <state_interface name="position"/>
+        <state_interface name="velocity"/>
+        <state_interface name="effort"/>
+        <param name="current_to_effort">2.20</param>
+      </joint>
+      <joint name="${NAME_JOINT_ARM_R_1}">
+        <command_interface name="position">
+          <param name="min">${JOINT_ARM_R_1_LOWER_LIMIT}</param>
+          <param name="max">${JOINT_ARM_R_1_UPPER_LIMIT}</param>
+        </command_interface>
+        <state_interface name="position"/>
+        <state_interface name="velocity"/>
+        <state_interface name="effort"/>
+        <param name="current_to_effort">3.60</param>
+      </joint>
+      <joint name="${NAME_JOINT_ARM_R_2}">
+        <command_interface name="position">
+          <param name="min">${JOINT_ARM_R_2_LOWER_LIMIT}</param>
+          <param name="max">${JOINT_ARM_R_2_UPPER_LIMIT}</param>
+        </command_interface>
+        <state_interface name="position"/>
+        <state_interface name="velocity"/>
+        <state_interface name="effort"/>
+        <param name="current_to_effort">3.60</param>
+      </joint>
+      <joint name="${NAME_JOINT_ARM_R_3}">
+        <command_interface name="position">
+          <param name="min">${JOINT_ARM_R_3_LOWER_LIMIT}</param>
+          <param name="max">${JOINT_ARM_R_3_UPPER_LIMIT}</param>
+        </command_interface>
+        <state_interface name="position"/>
+        <state_interface name="velocity"/>
+        <state_interface name="effort"/>
+        <param name="current_to_effort">2.20</param>
+      </joint>
+      <joint name="${NAME_JOINT_ARM_R_4}">
+        <command_interface name="position">
+          <param name="min">${JOINT_ARM_R_4_LOWER_LIMIT}</param>
+          <param name="max">${JOINT_ARM_R_4_UPPER_LIMIT}</param>
+        </command_interface>
+        <state_interface name="position"/>
+        <state_interface name="velocity"/>
+        <state_interface name="effort"/>
+        <param name="current_to_effort">2.00</param>
+      </joint>
+      <joint name="${NAME_JOINT_ARM_R_5}">
+        <command_interface name="position">
+          <param name="min">${JOINT_ARM_R_5_LOWER_LIMIT}</param>
+          <param name="max">${JOINT_ARM_R_5_UPPER_LIMIT}</param>
+        </command_interface>
+        <state_interface name="position"/>
+        <state_interface name="velocity"/>
+        <state_interface name="effort"/>
+        <param name="current_to_effort">2.20</param>
+      </joint>
+      <joint name="${NAME_JOINT_ARM_R_6}">
+        <command_interface name="position">
+          <param name="min">${JOINT_ARM_R_6_LOWER_LIMIT}</param>
+          <param name="max">${JOINT_ARM_R_6_UPPER_LIMIT}</param>
+        </command_interface>
+        <state_interface name="position"/>
+        <state_interface name="velocity"/>
+        <state_interface name="effort"/>
+        <param name="current_to_effort">2.20</param>
+      </joint>
+      <joint name="${NAME_JOINT_ARM_R_7}">
+        <command_interface name="position">
+          <param name="min">${JOINT_ARM_R_7_LOWER_LIMIT}</param>
+          <param name="max">${JOINT_ARM_R_7_UPPER_LIMIT}</param>
+        </command_interface>
+        <state_interface name="position"/>
+        <state_interface name="velocity"/>
+        <state_interface name="effort"/>
+        <param name="current_to_effort">2.20</param>
+      </joint>
+      <joint name="${NAME_JOINT_GRIPPER_R_A}">
+        <command_interface name="position">
+          <param name="min">${JOINT_GRIPPER_R_LOWER_LIMIT}</param>
+          <param name="max">${JOINT_GRIPPER_R_UPPER_LIMIT}</param>
+        </command_interface>
+        <state_interface name="position"/>
+        <state_interface name="velocity"/>
+        <state_interface name="effort"/>
+        <param name="current_to_effort">2.20</param>
+      </joint>
+      <joint name="${NAME_JOINT_ARM_L_1}">
+        <command_interface name="position">
+          <param name="min">${JOINT_ARM_L_1_LOWER_LIMIT}</param>
+          <param name="max">${JOINT_ARM_L_1_UPPER_LIMIT}</param>
+        </command_interface>
+        <state_interface name="position"/>
+        <state_interface name="velocity"/>
+        <state_interface name="effort"/>
+        <param name="current_to_effort">3.60</param>
+      </joint>
+      <joint name="${NAME_JOINT_ARM_L_2}">
+        <command_interface name="position">
+          <param name="min">${JOINT_ARM_L_2_LOWER_LIMIT}</param>
+          <param name="max">${JOINT_ARM_L_2_UPPER_LIMIT}</param>
+        </command_interface>
+        <state_interface name="position"/>
+        <state_interface name="velocity"/>
+        <state_interface name="effort"/>
+        <param name="current_to_effort">3.60</param>
+      </joint>
+      <joint name="${NAME_JOINT_ARM_L_3}">
+        <command_interface name="position">
+          <param name="min">${JOINT_ARM_L_3_LOWER_LIMIT}</param>
+          <param name="max">${JOINT_ARM_L_3_UPPER_LIMIT}</param>
+        </command_interface>
+        <state_interface name="position"/>
+        <state_interface name="velocity"/>
+        <state_interface name="effort"/>
+        <param name="current_to_effort">2.20</param>
+      </joint>
+      <joint name="${NAME_JOINT_ARM_L_4}">
+        <command_interface name="position">
+          <param name="min">${JOINT_ARM_L_4_LOWER_LIMIT}</param>
+          <param name="max">${JOINT_ARM_L_4_UPPER_LIMIT}</param>
+        </command_interface>
+        <state_interface name="position"/>
+        <state_interface name="velocity"/>
+        <state_interface name="effort"/>
+        <param name="current_to_effort">2.00</param>
+      </joint>
+      <joint name="${NAME_JOINT_ARM_L_5}">
+        <command_interface name="position">
+          <param name="min">${JOINT_ARM_L_5_LOWER_LIMIT}</param>
+          <param name="max">${JOINT_ARM_L_5_UPPER_LIMIT}</param>
+        </command_interface>
+        <state_interface name="position"/>
+        <state_interface name="velocity"/>
+        <state_interface name="effort"/>
+        <param name="current_to_effort">2.20</param>
+      </joint>
+      <joint name="${NAME_JOINT_ARM_L_6}">
+        <command_interface name="position">
+          <param name="min">${JOINT_ARM_L_6_LOWER_LIMIT}</param>
+          <param name="max">${JOINT_ARM_L_6_UPPER_LIMIT}</param>
+        </command_interface>
+        <state_interface name="position"/>
+        <state_interface name="velocity"/>
+        <state_interface name="effort"/>
+        <param name="current_to_effort">2.20</param>
+      </joint>
+      <joint name="${NAME_JOINT_ARM_L_7}">
+        <command_interface name="position">
+          <param name="min">${JOINT_ARM_L_7_LOWER_LIMIT}</param>
+          <param name="max">${JOINT_ARM_L_7_UPPER_LIMIT}</param>
+        </command_interface>
+        <state_interface name="position"/>
+        <state_interface name="velocity"/>
+        <state_interface name="effort"/>
+        <param name="current_to_effort">2.20</param>
+      </joint>
+      <joint name="${NAME_JOINT_GRIPPER_L_A}">
+        <command_interface name="position">
+          <param name="min">${JOINT_GRIPPER_L_LOWER_LIMIT}</param>
+          <param name="max">${JOINT_GRIPPER_L_UPPER_LIMIT}</param>
+        </command_interface>
+        <state_interface name="position"/>
+        <state_interface name="velocity"/>
+        <state_interface name="effort"/>
+        <param name="current_to_effort">2.20</param>
+      </joint>
+    </ros2_control>
+  </xacro:macro>
 </robot>

File: urdf/rakuda.xacro (robot description, xacro)
@@ -447,4 +447,5 @@
   <axis xyz="0.0 0.0 -1.0"/>
   <limit upper="1.396263" lower="-1.396263" effort="100" velocity="100"/>
+  <dynamics damping="1.0e-6" friction="0.8"/>
 </joint>
 <joint name="neck_yaw_joint" type="revolute">
@@ -454,4 +455,5 @@
   <axis xyz="0.0 0.0 1.0"/>
   <limit upper="1.22173" lower="-1.22173" effort="100" velocity="100"/>
+  <dynamics damping="1.0e-6" friction="0.8"/>
 </joint>
 <joint name="neck_pitch_joint" type="revolute">
@@ -461,4 +463,5 @@
   <axis xyz="0.0 -1.0 0.0"/>
   <limit upper="0.610865" lower="-0.872665" effort="100" velocity="100"/>
+  <dynamics damping="1.0e-6" friction="0.8"/>
 </joint>
 <joint name="l_arm_joint1" type="revolute">
@@ -468,4 +471,5 @@
   <axis xyz="0.0 1.0 0.0"/>
   <limit upper="0.0" lower="-2.96706" effort="100" velocity="100"/>
+  <dynamics damping="1.0e-6" friction="0.8"/>
 </joint>
 <joint name="r_arm_joint1" type="revolute">
@@ -475,4 +479,5 @@
   <axis xyz="0.0 -1.0 0.0"/>
   <limit upper="2.96706" lower="0.0" effort="100" velocity="100"/>
+  <dynamics damping="1.0e-6" friction="0.8"/>
 </joint>
 <joint name="l_arm_joint2" type="revolute">
@@ -482,4 +487,5 @@
   <axis xyz="1.0 0.0 0.0"/>
   <limit upper="1.570796" lower="-0.0" effort="100" velocity="100"/>
+  <dynamics damping="1.0e-6" friction="0.8"/>
 </joint>
 <joint name="r_arm_joint2" type="revolute">
@@ -489,4 +495,5 @@
   <axis xyz="1.0 0.0 0.0"/>
   <limit upper="0.0" lower="-1.570796" effort="100" velocity="100"/>
+  <dynamics damping="1.0e-6" friction="0.8"/>
 </joint>
 <joint name="l_arm_joint3" type="revolute">
@@ -496,4 +503,5 @@
   <axis xyz="0.0 0.0 -1.0"/>
   <limit upper="1.396263" lower="-1.396263" effort="100" velocity="100"/>
+  <dynamics damping="1.0e-6" friction="0.8"/>
 </joint>
 <joint name="r_arm_joint3" type="revolute">
@@ -503,4 +511,5 @@
   <axis xyz="0.0 0.0 -1.0"/>
   <limit upper="1.396263" lower="-1.396263" effort="100" velocity="100"/>
+  <dynamics damping="1.0e-6" friction="0.8"/>
 </joint>
 <joint name="l_arm_joint4" type="revolute">
@@ -510,4 +519,5 @@
   <axis xyz="0.0 1.0 0.0"/>
   <limit upper="0.174533" lower="-2.356194" effort="100" velocity="100"/>
+  <dynamics damping="1.0e-6" friction="0.8"/>
 </joint>
 <joint name="r_arm_joint4" type="revolute">
@@ -517,4 +527,5 @@
   <axis xyz="0.0 -1.0 0.0"/>
   <limit upper="2.356194" lower="-0.174533" effort="100" velocity="100"/>
+  <dynamics damping="1.0e-6" friction="0.8"/>
 </joint>
 <joint name="l_arm_joint5" type="revolute">
@@ -524,4 +535,5 @@
   <axis xyz="0.0 0.0 -1.0"/>
   <limit upper="1.570796" lower="-1.570796" effort="100" velocity="100"/>
+  <dynamics damping="1.0e-6" friction="0.8"/>
 </joint>
 <joint name="r_arm_joint5" type="revolute">
@@ -531,4 +543,5 @@
   <axis xyz="0.0 0.0 -1.0"/>
   <limit upper="1.570796" lower="-1.570796" effort="100" velocity="100"/>
+  <dynamics damping="1.0e-6" friction="0.8"/>
 </joint>
 <joint name="r_arm_joint6" type="revolute">
@@ -538,4 +551,5 @@
   <axis xyz="0.0 -1.0 0.0"/>
   <limit upper="1.396263" lower="-1.396263" effort="100" velocity="100"/>
+  <dynamics damping="1.0e-6" friction="0.8"/>
 </joint>
 <joint name="l_arm_joint6" type="revolute">
@@ -545,4 +559,5 @@
   <axis xyz="0.0 1.0 0.0"/>
   <limit upper="1.396263" lower="-1.396263" effort="100" velocity="100"/>
+  <dynamics damping="1.0e-6" friction="0.8"/>
 </joint>
 <joint name="r_gripper_joint" type="revolute">
@@ -552,4 +567,5 @@
   <axis xyz="1.0 0.0 0.0"/>
   <limit upper="0.0" lower="-1.22173" effort="100" velocity="100"/>
+  <dynamics damping="1.0e-6" friction="0.8"/>
 </joint>
 <joint name="r_gripper_mimic_joint" type="revolute">
@@ -567,4 +583,5 @@
   <axis xyz="1.0 0.0 0.0"/>
   <limit upper="1.22173" lower="0.0" effort="100" velocity="100"/>
+  <dynamics damping="1.0e-6" friction="0.8"/>
 </joint>
 <joint name="l_gripper_mimic_joint" type="revolute">
