Commit message: feat: update DOF value to 17 in rakuda.xacro for enhanced robot control

File: urdf/rakuda.ros2_control.xacro (robot description, xacro)
@@ -81,4 +81,39 @@
         <state_interface name="effort"/>
       </joint>
+      <joint name="r_arm_joint1">
+        <state_interface name="position"/>
+        <state_interface name="velocity"/>
+        <state_interface name="effort"/>
+      </joint>
+      <joint name="r_arm_joint2">
+        <state_interface name="position"/>
+        <state_interface name="velocity"/>
+        <state_interface name="effort"/>
+      </joint>
+      <joint name="r_arm_joint3">
+        <state_interface name="position"/>
+        <state_interface name="velocity"/>
+        <state_interface name="effort"/>
+      </joint>
+      <joint name="r_arm_joint4">
+        <state_interface name="position"/>
+        <state_interface name="velocity"/>
+        <state_interface name="effort"/>
+      </joint>
+      <joint name="r_arm_joint5">
+        <state_interface name="position"/>
+        <state_interface name="velocity"/>
+        <state_interface name="effort"/>
+      </joint>
+      <joint name="r_arm_joint6">
+        <state_interface name="position"/>
+        <state_interface name="velocity"/>
+        <state_interface name="effort"/>
+      </joint>
+      <joint name="r_gripper_joint">
+        <state_interface name="position"/>
+        <state_interface name="velocity"/>
+        <state_interface name="effort"/>
+      </joint>
 <!--TORSO -->
       <gpio name="dxl1">
@@ -238,4 +273,109 @@
       </gpio>
 <!--RIGHT ARM -->
+      <gpio name="dxl21">
+        <param name="type">dxl</param>
+        <param name="ID">21</param>
+        <state_interface name="Present Position"/>
+        <state_interface name="Present Velocity"/>
+        <!--<state_interface name="Present Current"/> -->
+        <param name="Operating Mode">3</param>
+        <param name="Profile Velocity">40</param>
+        <param name="Profile Acceleration">20</param>
+        <param name="Position P Gain">800</param>
+        <param name="Position I Gain">100</param>
+        <param name="Position D Gain">100</param>
+        <param name="Return Delay Time">0</param>
+        <param name="Drive Mode">0</param>
+      </gpio>
+      <gpio name="dxl22">
+        <param name="type">dxl</param>
+        <param name="ID">22</param>
+        <state_interface name="Present Position"/>
+        <state_interface name="Present Velocity"/>
+        <!--<state_interface name="Present Current"/> -->
+        <param name="Operating Mode">3</param>
+        <param name="Profile Velocity">40</param>
+        <param name="Profile Acceleration">20</param>
+        <param name="Position P Gain">800</param>
+        <param name="Position I Gain">100</param>
+        <param name="Position D Gain">100</param>
+        <param name="Return Delay Time">0</param>
+        <param name="Drive Mode">1</param>
+      </gpio>
+      <gpio name="dxl23">
+        <param name="type">dxl</param>
+        <param name="ID">23</param>
+        <state_interface name="Present Position"/>
+        <state_interface name="Present Velocity"/>
+        <!--<state_interface name="Present Current"/> -->
+        <param name="Operating Mode">3</param>
+        <param name="Profile Velocity">40</param>
+        <param name="Profile Acceleration">20</param>
+        <param name="Position P Gain">800</param>
+        <param name="Position I Gain">100</param>
+        <param name="Position D Gain">100</param>
+        <param name="Return Delay Time">0</param>
+        <param name="Drive Mode">0</param>
+      </gpio>
+      <gpio name="dxl24">
+        <param name="type">dxl</param>
+        <param name="ID">24</param>
+        <state_interface name="Present Position"/>
+        <state_interface name="Present Velocity"/>
+        <!--<state_interface name="Present Current"/> -->
+        <param name="Operating Mode">3</param>
+        <param name="Profile Velocity">40</param>
+        <param name="Profile Acceleration">20</param>
+        <param name="Position P Gain">800</param>
+        <param name="Position I Gain">100</param>
+        <param name="Position D Gain">100</param>
+        <param name="Return Delay Time">0</param>
+        <param name="Drive Mode">0</param>
+      </gpio>
+      <gpio name="dxl25">
+        <param name="type">dxl</param>
+        <param name="ID">25</param>
+        <state_interface name="Present Position"/>
+        <state_interface name="Present Velocity"/>
+        <!--<state_interface name="Present Current"/> -->
+        <param name="Operating Mode">3</param>
+        <param name="Profile Velocity">40</param>
+        <param name="Profile Acceleration">20</param>
+        <param name="Position P Gain">800</param>
+        <param name="Position I Gain">100</param>
+        <param name="Position D Gain">100</param>
+        <param name="Return Delay Time">0</param>
+        <param name="Drive Mode">0</param>
+      </gpio>
+      <gpio name="dxl26">
+        <param name="type">dxl</param>
+        <param name="ID">26</param>
+        <state_interface name="Present Position"/>
+        <state_interface name="Present Velocity"/>
+        <!--<state_interface name="Present Current"/> -->
+        <param name="Operating Mode">3</param>
+        <param name="Profile Velocity">40</param>
+        <param name="Profile Acceleration">20</param>
+        <param name="Position P Gain">800</param>
+        <param name="Position I Gain">100</param>
+        <param name="Position D Gain">100</param>
+        <param name="Return Delay Time">0</param>
+        <param name="Drive Mode">0</param>
+      </gpio>
+      <gpio name="dxl27">
+        <param name="type">dxl</param>
+        <param name="ID">27</param>
+        <state_interface name="Present Position"/>
+        <state_interface name="Present Velocity"/>
+        <!--<state_interface name="Present Current"/> -->
+        <param name="Operating Mode">3</param>
+        <param name="Profile Velocity">40</param>
+        <param name="Profile Acceleration">20</param>
+        <param name="Position P Gain">800</param>
+        <param name="Position I Gain">100</param>
+        <param name="Position D Gain">100</param>
+        <param name="Return Delay Time">0</param>
+        <param name="Drive Mode">0</param>
+      </gpio>
     </ros2_control>
   </xacro:macro>

File: urdf/rakuda.xacro (robot description, xacro)
@@ -115,5 +115,5 @@
 <xacro:gemini_335_336 parent_link="neck_pitch_link" />
 <!-- Chiama la macro che aggancia il ros control: Inserire il numero di Dynamixel -->
-<xacro:property name="dof" value="10"/>
+<xacro:property name="dof" value="17"/>
 <xacro:include filename="rakuda.ros2_control.xacro"/>
 <xacro:rakuda_ros2_control_settings dof="${dof}"/>

Commit message: bug fixes

File: urdf/rakuda.ros2_control.xacro (robot description, xacro)
@@ -83,4 +83,5 @@
       </joint>
       <joint name="l_gripper_joint">
+      	<command_interface name="position"/>
         <state_interface name="position"/>
         <state_interface name="velocity"/>
@@ -124,4 +125,5 @@
       </joint>
       <joint name="r_gripper_joint">
+      	<command_interface name="position"/>
         <state_interface name="position"/>
         <state_interface name="velocity"/>
@@ -135,5 +137,5 @@
         <state_interface name="Present Position"/>
         <state_interface name="Present Velocity"/>
-        <!--<state_interface name="Present Current"/> -->
+        <state_interface name="Present Current"/>
         <param name="Operating Mode">3</param>
         <param name="Profile Velocity">40</param>
@@ -187,6 +189,6 @@
         <!--<state_interface name="Present Current"/> -->
         <param name="Operating Mode">3</param>
-        <param name="Profile Velocity">40</param>
-        <param name="Profile Acceleration">20</param>
+        <param name="Profile Velocity">80</param>
+        <param name="Profile Acceleration">40</param>
         <param name="Position P Gain">800</param>
         <param name="Position I Gain">100</param>
@@ -203,6 +205,6 @@
         <!--<state_interface name="Present Current"/> -->
         <param name="Operating Mode">3</param>
-        <param name="Profile Velocity">40</param>
-        <param name="Profile Acceleration">20</param>
+        <param name="Profile Velocity">80</param>
+        <param name="Profile Acceleration">40</param>
         <param name="Position P Gain">800</param>
         <param name="Position I Gain">100</param>
@@ -219,6 +221,6 @@
         <!--<state_interface name="Present Current"/> -->
         <param name="Operating Mode">3</param>
-        <param name="Profile Velocity">40</param>
-        <param name="Profile Acceleration">20</param>
+        <param name="Profile Velocity">80</param>
+        <param name="Profile Acceleration">40</param>
         <param name="Position P Gain">800</param>
         <param name="Position I Gain">100</param>
@@ -235,6 +237,6 @@
         <!--<state_interface name="Present Current"/> -->
         <param name="Operating Mode">3</param>
-        <param name="Profile Velocity">40</param>
-        <param name="Profile Acceleration">20</param>
+        <param name="Profile Velocity">80</param>
+        <param name="Profile Acceleration">40</param>
         <param name="Position P Gain">800</param>
         <param name="Position I Gain">100</param>
@@ -251,6 +253,6 @@
         <!--<state_interface name="Present Current"/> -->
         <param name="Operating Mode">3</param>
-        <param name="Profile Velocity">40</param>
-        <param name="Profile Acceleration">20</param>
+        <param name="Profile Velocity">80</param>
+        <param name="Profile Acceleration">40</param>
         <param name="Position P Gain">800</param>
         <param name="Position I Gain">100</param>
@@ -260,5 +262,4 @@
       </gpio>
       <gpio name="dxl16">
-      <command_interface name="Goal Position"/>
         <param name="type">dxl</param>
         <param name="ID">16</param>
@@ -268,6 +269,6 @@
         <!--<state_interface name="Present Current"/> -->
         <param name="Operating Mode">3</param>
-        <param name="Profile Velocity">40</param>
-        <param name="Profile Acceleration">20</param>
+        <param name="Profile Velocity">80</param>
+        <param name="Profile Acceleration">40</param>
         <param name="Position P Gain">800</param>
         <param name="Position I Gain">100</param>
@@ -279,10 +280,11 @@
         <param name="type">dxl</param>
         <param name="ID">17</param>
-        <state_interface name="Present Position"/>
-        <state_interface name="Present Velocity"/>
-        <!--<state_interface name="Present Current"/> -->
-        <param name="Operating Mode">3</param>
-        <param name="Profile Velocity">40</param>
-        <param name="Profile Acceleration">20</param>
+        <command_interface name="Goal Position"/>
+        <state_interface name="Present Position"/>
+        <state_interface name="Present Velocity"/>
+        <!--<state_interface name="Present Current"/> -->
+        <param name="Operating Mode">3</param>
+        <param name="Profile Velocity">100</param>
+        <param name="Profile Acceleration">40</param>
         <param name="Position P Gain">800</param>
         <param name="Position I Gain">100</param>
@@ -300,6 +302,6 @@
         <!--<state_interface name="Present Current"/> -->
         <param name="Operating Mode">3</param>
-        <param name="Profile Velocity">40</param>
-        <param name="Profile Acceleration">20</param>
+        <param name="Profile Velocity">80</param>
+        <param name="Profile Acceleration">40</param>
         <param name="Position P Gain">800</param>
         <param name="Position I Gain">100</param>
@@ -316,6 +318,6 @@
         <!--<state_interface name="Present Current"/> -->
         <param name="Operating Mode">3</param>
-        <param name="Profile Velocity">40</param>
-        <param name="Profile Acceleration">20</param>
+        <param name="Profile Velocity">80</param>
+        <param name="Profile Acceleration">40</param>
         <param name="Position P Gain">800</param>
         <param name="Position I Gain">100</param>
@@ -332,6 +334,6 @@
         <!--<state_interface name="Present Current"/> -->
         <param name="Operating Mode">3</param>
-        <param name="Profile Velocity">40</param>
-        <param name="Profile Acceleration">20</param>
+        <param name="Profile Velocity">80</param>
+        <param name="Profile Acceleration">40</param>
         <param name="Position P Gain">800</param>
         <param name="Position I Gain">100</param>
@@ -348,6 +350,6 @@
         <!--<state_interface name="Present Current"/> -->
         <param name="Operating Mode">3</param>
-        <param name="Profile Velocity">40</param>
-        <param name="Profile Acceleration">20</param>
+        <param name="Profile Velocity">80</param>
+        <param name="Profile Acceleration">40</param>
         <param name="Position P Gain">800</param>
         <param name="Position I Gain">100</param>
@@ -364,6 +366,6 @@
         <!--<state_interface name="Present Current"/> -->
         <param name="Operating Mode">3</param>
-        <param name="Profile Velocity">40</param>
-        <param name="Profile Acceleration">20</param>
+        <param name="Profile Velocity">80</param>
+        <param name="Profile Acceleration">40</param>
         <param name="Position P Gain">800</param>
         <param name="Position I Gain">100</param>
@@ -380,6 +382,6 @@
         <!--<state_interface name="Present Current"/> -->
         <param name="Operating Mode">3</param>
-        <param name="Profile Velocity">40</param>
-        <param name="Profile Acceleration">20</param>
+        <param name="Profile Velocity">80</param>
+        <param name="Profile Acceleration">40</param>
         <param name="Position P Gain">800</param>
         <param name="Position I Gain">100</param>
@@ -391,10 +393,11 @@
         <param name="type">dxl</param>
         <param name="ID">27</param>
-        <state_interface name="Present Position"/>
-        <state_interface name="Present Velocity"/>
-        <!--<state_interface name="Present Current"/> -->
-        <param name="Operating Mode">3</param>
-        <param name="Profile Velocity">40</param>
-        <param name="Profile Acceleration">20</param>
+        <command_interface name="Goal Position"/>
+        <state_interface name="Present Position"/>
+        <state_interface name="Present Velocity"/>
+        <!--<state_interface name="Present Current"/> -->
+        <param name="Operating Mode">3</param>
+        <param name="Profile Velocity">100</param>
+        <param name="Profile Acceleration">40</param>
         <param name="Position P Gain">800</param>
         <param name="Position I Gain">100</param>

File: urdf/rakuda.xacro (robot description, xacro)
@@ -448,5 +448,5 @@
   <child link="torso_link"/>
   <axis xyz="0.0 0.0 1.0"/>
-  <limit upper="1.396263" lower="-1.396263" effort="100" velocity="100"/>
+  <limit upper="1.396263" lower="-1.396263" effort="100.0" velocity="4.8"/>
   <dynamics damping="1.0e-6" friction="0.8"/>
 </joint>
@@ -456,6 +456,6 @@
   <child link="neck_yaw_link"/>
   <axis xyz="0.0 0.0 1.0"/>
-  <!-- Sciurus17 limit upper="1.22173" lower="-1.22173" effort="100" velocity="100"/ -->
-  <limit upper="0.660" lower="-0.660" effort="100" velocity="100"/>
+  <!-- Sciurus17 limit upper="1.22173" lower="-1.22173" effort="100.0" velocity="4.8"/ -->
+  <limit upper="0.660" lower="-0.660" effort="100.0" velocity="4.8"/>
   <dynamics damping="1.0e-6" friction="0.8"/>
 </joint>
@@ -465,5 +465,5 @@
   <child link="l_link1"/>
   <axis xyz="0.0 1.0 0.0"/>
-  <limit upper="0.0" lower="-2.96706" effort="100" velocity="100"/>
+  <limit upper="0.0" lower="-2.96706" effort="100.0" velocity="4.8"/>
   <dynamics damping="1.0e-6" friction="0.8"/>
 </joint>
@@ -473,5 +473,5 @@
   <child link="r_link1"/>
   <axis xyz="0.0 -1.0 0.0"/>
-  <limit upper="2.96706" lower="0.0" effort="100" velocity="100"/>
+  <limit upper="2.96706" lower="0.0" effort="100.0" velocity="4.8"/>
   <dynamics damping="1.0e-6" friction="0.8"/>
 </joint>
@@ -481,5 +481,5 @@
   <child link="l_link2"/>
   <axis xyz="1.0 0.0 0.0"/>
-  <limit upper="1.570796" lower="-0.0" effort="100" velocity="100"/>
+  <limit upper="1.570796" lower="-0.0" effort="100.0" velocity="4.8"/>
   <dynamics damping="1.0e-6" friction="0.8"/>
 </joint>
@@ -489,5 +489,5 @@
   <child link="r_link2"/>
   <axis xyz="1.0 0.0 0.0"/>
-  <limit upper="0.0" lower="-1.570796" effort="100" velocity="100"/>
+  <limit upper="0.0" lower="-1.570796" effort="100.0" velocity="4.8"/>
   <dynamics damping="1.0e-6" friction="0.8"/>
 </joint>
@@ -497,5 +497,5 @@
   <child link="l_link3"/>
   <axis xyz="0.0 0.0 -1.0"/>
-  <limit upper="1.396263" lower="-1.396263" effort="100" velocity="100"/>
+  <limit upper="1.396263" lower="-1.396263" effort="100.0" velocity="4.8"/>
   <dynamics damping="1.0e-6" friction="0.8"/>
 </joint>
@@ -505,5 +505,5 @@
   <child link="r_link3"/>
   <axis xyz="0.0 0.0 -1.0"/>
-  <limit upper="1.396263" lower="-1.396263" effort="100" velocity="100"/>
+  <limit upper="1.396263" lower="-1.396263" effort="100.0" velocity="4.8"/>
   <dynamics damping="1.0e-6" friction="0.8"/>
 </joint>
@@ -513,5 +513,5 @@
   <child link="l_link4"/>
   <axis xyz="0.0 1.0 0.0"/>
-  <limit upper="0.174533" lower="-2.356194" effort="100" velocity="100"/>
+  <limit upper="0.174533" lower="-2.356194" effort="100.0" velocity="4.8"/>
   <dynamics damping="1.0e-6" friction="0.8"/>
 </joint>
@@ -521,5 +521,5 @@
   <child link="r_link4"/>
   <axis xyz="0.0 -1.0 0.0"/>
-  <limit upper="2.356194" lower="-0.174533" effort="100" velocity="100"/>
+  <limit upper="2.356194" lower="-0.174533" effort="100.0" velocity="4.8"/>
   <dynamics damping="1.0e-6" friction="0.8"/>
 </joint>
@@ -529,5 +529,5 @@
   <child link="l_link5"/>
   <axis xyz="0.0 0.0 -1.0"/>
-  <limit upper="1.570796" lower="-1.570796" effort="100" velocity="100"/>
+  <limit upper="1.570796" lower="-1.570796" effort="100.0" velocity="4.8"/>
   <dynamics damping="1.0e-6" friction="0.8"/>
 </joint>
@@ -537,5 +537,5 @@
   <child link="r_link5"/>
   <axis xyz="0.0 0.0 -1.0"/>
-  <limit upper="1.570796" lower="-1.570796" effort="100" velocity="100"/>
+  <limit upper="1.570796" lower="-1.570796" effort="100.0" velocity="4.8"/>
   <dynamics damping="1.0e-6" friction="0.8"/>
 </joint>
@@ -545,5 +545,5 @@
   <child link="r_link6"/>
   <axis xyz="0.0 -1.0 0.0"/>
-  <limit upper="1.396263" lower="-1.396263" effort="100" velocity="100"/>
+  <limit upper="1.396263" lower="-1.396263" effort="100.0" velocity="4.8"/>
   <dynamics damping="1.0e-6" friction="0.8"/>
 </joint>
@@ -553,5 +553,5 @@
   <child link="l_link6"/>
   <axis xyz="0.0 1.0 0.0"/>
-  <limit upper="1.396263" lower="-1.396263" effort="100" velocity="100"/>
+  <limit upper="1.396263" lower="-1.396263" effort="100.0" velocity="4.8"/>
   <dynamics damping="1.0e-6" friction="0.8"/>
 </joint>
@@ -561,5 +561,5 @@
   <child link="r_gripper_a"/>
   <axis xyz="1.0 0.0 0.0"/>
-  <limit upper="0.0" lower="-1.22173" effort="100" velocity="100"/>
+  <limit upper="0.0" lower="-1.22173" effort="100.0" velocity="4.8"/>
   <dynamics damping="1.0e-6" friction="0.8"/>
 </joint>
@@ -577,5 +577,5 @@
   <child link="l_gripper_a"/>
   <axis xyz="1.0 0.0 0.0"/>
-  <limit upper="1.22173" lower="0.0" effort="100" velocity="100"/>
+  <limit upper="1.22173" lower="0.0" effort="100.0" velocity="4.8"/>
   <dynamics damping="1.0e-6" friction="0.8"/>
 </joint>
