Commit message: cleansed

File: urdf/rakuda.ros2_control.xacro (robot description, xacro)
@@ -1,4 +1,34 @@
 <?xml version="1.0"?>
 <robot xmlns:xacro="http://www.ros.org/wiki/xacro">
+  <!--
+  ╔═════════════════════════════════════════════════════════════════════╗
+  ║           MAPPING JOINT <-> DYNAMIXEL  (transmission matrix)        ║
+  ║  Index   │ Nome joint          │ gpio name              │ ID        ║
+  ║──────────┼─────────────────────┼────────────────────────┼───────────║
+  ║  0       │ waist_yaw_joint     │ waist_yaw_dxl          │  1        ║
+  ║  1       │ neck_yaw_joint      │ neck_yaw_dxl           │  2        ║
+  ║  2       │ neck_pitch_joint    │ neck_pitch_dxl         │  3        ║
+  ║  3       │ l_arm_joint1        │ l_arm_joint1_dxl       │ 11        ║
+  ║  4       │ l_arm_joint2        │ l_arm_joint2_dxl       │ 12        ║
+  ║  5       │ l_arm_joint3        │ l_arm_joint3_dxl       │ 13        ║
+  ║  6       │ l_arm_joint4        │ l_arm_joint4_dxl       │ 14        ║
+  ║  7       │ l_arm_joint5        │ l_arm_joint5_dxl       │ 15        ║
+  ║  8       │ l_arm_joint6        │ l_arm_joint6_dxl       │ 16        ║
+  ║  9       │ l_gripper_joint     │ l_gripper_dxl          │ 17        ║
+  ║ 10       │ r_arm_joint1        │ r_arm_joint1_dxl       │ 21        ║
+  ║ 11       │ r_arm_joint2        │ r_arm_joint2_dxl       │ 22        ║
+  ║ 12       │ r_arm_joint3        │ r_arm_joint3_dxl       │ 23        ║
+  ║ 13       │ r_arm_joint4        │ r_arm_joint4_dxl       │ 24        ║
+  ║ 14       │ r_arm_joint5        │ r_arm_joint5_dxl       │ 25        ║
+  ║ 15       │ r_arm_joint6        │ r_arm_joint6_dxl       │ 26        ║
+  ║ 16       │ r_gripper_joint     │ r_gripper_dxl          │ 27        ║
+  ╚═════════════════════════════════════════════════════════════════════╝
+  NOTA: i gpio devono essere dichiarati nello STESSO ORDINE degli indici
+  della tabella, perché la transmission matrix identità mappa joint[i] <-> gpio[i].
+  NON riordinare i blocchi gpio senza aggiornare anche la tabella sopra.
+  NOTA: Present Current è commentato intenzionalmente su tutti i motori
+  tranne dxl1 (torso). Sarà abilitato in futuro per la gravity compensation.
+  Drive Mode: 0 = normale (CW), 1 = invertito (CCW)
+  -->
   <!-- Crea la matrice identità NxN Dynamixel -->
   <xacro:macro name="identity_matrix_csv" params="n">
@@ -9,6 +39,5 @@
     ])}
   </xacro:macro>
-<xacro:macro name="rakuda_ros2_control_settings" params="dof use_mock_hardware:=true mock_sensor_commands:=true">
-  <!-- (consiglio) rinomina per non confondere i log -->
+<xacro:macro name="rakuda_ros2_control_settings" params="dof use_mock_hardware:=false mock_sensor_commands:=false">
   <ros2_control name="RakudaSystem" type="system">
     <hardware>
@@ -35,4 +64,6 @@
         </xacro:unless>
       </hardware>
+<!-- JOINT INTERFACE (ros2_control / moveit)-->
+      <!-- index 0 -->
       <joint name="waist_yaw_joint">
         <command_interface name="position"/>
@@ -41,4 +72,5 @@
         <state_interface name="effort"/>
       </joint>
+      <!-- index 1 -->
       <joint name="neck_yaw_joint">
         <command_interface name="position"/>
@@ -47,4 +79,5 @@
         <state_interface name="effort"/>
       </joint>
+      <!-- index 2 -->
       <joint name="neck_pitch_joint">
         <command_interface name="position"/>
@@ -53,4 +86,5 @@
         <state_interface name="effort"/>
       </joint>
+      <!-- index 3 -->
       <joint name="l_arm_joint1">
         <command_interface name="position"/>
@@ -59,4 +93,5 @@
         <state_interface name="effort"/>
       </joint>
+      <!-- index 4 -->
       <joint name="l_arm_joint2">
         <command_interface name="position"/>
@@ -65,4 +100,5 @@
         <state_interface name="effort"/>
       </joint>
+      <!-- index 5 -->
       <joint name="l_arm_joint3">
         <command_interface name="position"/>
@@ -71,4 +107,5 @@
         <state_interface name="effort"/>
       </joint>
+      <!-- index 6 -->
       <joint name="l_arm_joint4">
         <command_interface name="position"/>
@@ -77,4 +114,5 @@
         <state_interface name="effort"/>
       </joint>
+      <!-- index 7 -->
       <joint name="l_arm_joint5">
         <command_interface name="position"/>
@@ -83,4 +121,5 @@
         <state_interface name="effort"/>
       </joint>
+      <!-- index 8 -->
       <joint name="l_arm_joint6">
         <command_interface name="position"/>
@@ -89,4 +128,5 @@
         <state_interface name="effort"/>
       </joint>
+      <!-- index 9 -->
       <joint name="l_gripper_joint">
       	<command_interface name="position"/>
@@ -95,4 +135,5 @@
         <state_interface name="effort"/>
       </joint>
+      <!-- index 10 -->
       <joint name="r_arm_joint1">
         <command_interface name="position"/>
@@ -101,4 +142,5 @@
         <state_interface name="effort"/>
       </joint>
+      <!-- index 11 -->
       <joint name="r_arm_joint2">
         <command_interface name="position"/>
@@ -107,4 +149,5 @@
         <state_interface name="effort"/>
       </joint>
+      <!-- index 12 -->
       <joint name="r_arm_joint3">
         <command_interface name="position"/>
@@ -113,4 +156,5 @@
         <state_interface name="effort"/>
       </joint>
+      <!-- index 13 -->
       <joint name="r_arm_joint4">
         <command_interface name="position"/>
@@ -119,4 +163,5 @@
         <state_interface name="effort"/>
       </joint>
+      <!-- index 14 -->
       <joint name="r_arm_joint5">
         <command_interface name="position"/>
@@ -125,4 +170,5 @@
         <state_interface name="effort"/>
       </joint>
+      <!-- index 15 -->
       <joint name="r_arm_joint6">
         <command_interface name="position"/>
@@ -131,4 +177,5 @@
         <state_interface name="effort"/>
       </joint>
+      <!-- index 16 -->
       <joint name="r_gripper_joint">
       	<command_interface name="position"/>
@@ -137,6 +184,8 @@
         <state_interface name="effort"/>
       </joint>
+<!-- GPIO /Dynamixel Hardware -->
 <!--TORSO -->
-      <gpio name="dxl1">
+      <!-- index 0 | waist_yaw_joint | ID 1 -->
+      <gpio name="waist_yaw_dxl">
         <param name="type">dxl</param>
         <param name="ID">1</param>
@@ -155,5 +204,6 @@
       </gpio>
 <!--HEAD -->
-      <gpio name="dxl2">
+      <!-- index 1 | neck_yaw_joint | ID 2 -->
+      <gpio name="neck_yaw_dxl">
         <param name="type">dxl</param>
         <param name="ID">2</param>
@@ -171,5 +221,6 @@
         <param name="Drive Mode">0</param>
       </gpio>
-      <gpio name="dxl3">
+      <!-- index 2 | neck_pitch_joint | ID 3 | Drive Mode 1 = invertito -->
+      <gpio name="neck_pitch_dxl">
         <param name="type">dxl</param>
         <param name="ID">3</param>
@@ -188,5 +239,6 @@
       </gpio>
 <!--LEFT ARM -->
-      <gpio name="dxl11">
+      <!-- index 3 | l_arm_joint1 | ID 11 -->
+      <gpio name="l_arm_joint1_dxl">
         <param name="type">dxl</param>
         <param name="ID">11</param>
@@ -204,5 +256,6 @@
         <param name="Drive Mode">0</param>
       </gpio>
-      <gpio name="dxl12">
+      <!-- index 4 | l_arm_joint2 | ID 12 | Drive Mode 1 = invertito -->
+      <gpio name="l_arm_joint2_dxl">
         <param name="type">dxl</param>
         <param name="ID">12</param>
@@ -220,5 +273,6 @@
         <param name="Drive Mode">1</param>
       </gpio>
-      <gpio name="dxl13">
+      <!-- index 5 | l_arm_joint3 | ID 13 -->
+      <gpio name="l_arm_joint3_dxl">
         <param name="type">dxl</param>
         <param name="ID">13</param>
@@ -236,5 +290,6 @@
         <param name="Drive Mode">0</param>
       </gpio>
-      <gpio name="dxl14">
+      <!-- index 6 | l_arm_joint4 | ID 14 -->
+      <gpio name="l_arm_joint4_dxl">
         <param name="type">dxl</param>
         <param name="ID">14</param>
@@ -252,5 +307,6 @@
         <param name="Drive Mode">0</param>
       </gpio>
-      <gpio name="dxl15">
+      <!-- index 7 | l_arm_joint5 | ID 15 -->
+      <gpio name="l_arm_joint5_dxl">
         <param name="type">dxl</param>
         <param name="ID">15</param>
@@ -268,5 +324,6 @@
         <param name="Drive Mode">0</param>
       </gpio>
-      <gpio name="dxl16">
+      <!-- index 8 | l_arm_joint6 | ID 16 -->
+      <gpio name="l_arm_joint6_dxl">
         <param name="type">dxl</param>
         <param name="ID">16</param>
@@ -284,5 +341,6 @@
         <param name="Drive Mode">0</param>
       </gpio>
-      <gpio name="dxl17">
+      <!-- index 9 | l_gripper_joint | ID 17 -->
+      <gpio name="l_gripper_dxl">
         <param name="type">dxl</param>
         <param name="ID">17</param>
@@ -301,5 +359,6 @@
       </gpio>
 <!--RIGHT ARM -->
-      <gpio name="dxl21">
+      <!-- index 10 | r_arm_joint1 | ID 21 -->
+      <gpio name="r_arm_joint1_dxl">
         <param name="type">dxl</param>
         <param name="ID">21</param>
@@ -317,5 +376,6 @@
         <param name="Drive Mode">0</param>
       </gpio>
-      <gpio name="dxl22">
+      <!-- index 11 | r_arm_joint2 | ID 22 | Drive Mode 1 = invertito -->
+      <gpio name="r_arm_joint2_dxl">
         <param name="type">dxl</param>
         <param name="ID">22</param>
@@ -333,5 +393,6 @@
         <param name="Drive Mode">1</param>
       </gpio>
-      <gpio name="dxl23">
+      <!-- index 12 | r_arm_joint3 | ID 23 -->
+      <gpio name="r_arm_joint3_dxl">
         <param name="type">dxl</param>
         <param name="ID">23</param>
@@ -349,5 +410,6 @@
         <param name="Drive Mode">0</param>
       </gpio>
-      <gpio name="dxl24">
+      <!-- index 13 | r_arm_joint4 | ID 24 -->
+      <gpio name="r_arm_joint4_dxl">
         <param name="type">dxl</param>
         <param name="ID">24</param>
@@ -365,5 +427,6 @@
         <param name="Drive Mode">0</param>
       </gpio>
-      <gpio name="dxl25">
+      <!-- index 14 | r_arm_joint5 | ID 25 -->
+      <gpio name="r_arm_joint5_dxl">
         <param name="type">dxl</param>
         <param name="ID">25</param>
@@ -381,5 +444,6 @@
         <param name="Drive Mode">0</param>
       </gpio>
-      <gpio name="dxl26">
+      <!-- index 15 | r_arm_joint6 | ID 26 -->
+      <gpio name="r_arm_joint6_dxl">
         <param name="type">dxl</param>
         <param name="ID">26</param>
@@ -397,5 +461,6 @@
         <param name="Drive Mode">0</param>
       </gpio>
-      <gpio name="dxl27">
+      <!-- index 16 | r_gripper_joint | ID 27 -->
+      <gpio name="r_gripper_dxl">
         <param name="type">dxl</param>
         <param name="ID">27</param>

Commit message: tuning of joint limits

File: urdf/rakuda.ros2_control.xacro (robot description, xacro)
@@ -184,4 +184,5 @@
         <state_interface name="effort"/>
       </joint>
+      <xacro:unless value="${use_mock_hardware}">
 <!-- GPIO /Dynamixel Hardware -->
 <!--TORSO -->
@@ -478,4 +479,5 @@
         <param name="Drive Mode">0</param>
       </gpio>
+      </xacro:unless>
     </ros2_control>
   </xacro:macro>

File: urdf/rakuda.urdf.xacro (robot description, xacro)
@@ -469,5 +469,5 @@
   <child link="l_link1"/>
   <axis xyz="0.0 1.0 0.0"/>
-  <limit upper="0.0" lower="-2.96706" effort="10.0" velocity="4.8"/>
+  <limit upper="0.250" lower="-2.96706" effort="10.0" velocity="4.8"/>
   <dynamics damping="1.0e-6" friction="0.8"/>
 </joint>
@@ -477,5 +477,5 @@
   <child link="r_link1"/>
   <axis xyz="0.0 -1.0 0.0"/>
-  <limit upper="2.96706" lower="0.0" effort="10.0" velocity="4.8"/>
+  <limit upper="2.96706" lower="-0.250" effort="10.0" velocity="4.8"/>
   <dynamics damping="1.0e-6" friction="0.8"/>
 </joint>
@@ -485,5 +485,5 @@
   <child link="l_link2"/>
   <axis xyz="1.0 0.0 0.0"/>
-  <limit upper="1.570796" lower="-0.0" effort="10.0" velocity="4.8"/>
+  <limit upper="1.570796" lower="-0.2" effort="10.0" velocity="4.8"/>
   <dynamics damping="1.0e-6" friction="0.8"/>
 </joint>
@@ -493,5 +493,5 @@
   <child link="r_link2"/>
   <axis xyz="1.0 0.0 0.0"/>
-  <limit upper="0.0" lower="-1.570796" effort="10.0" velocity="4.8"/>
+  <limit upper="0.2" lower="-1.570796" effort="10.0" velocity="4.8"/>
   <dynamics damping="1.0e-6" friction="0.8"/>
 </joint>
